Commit message: Style fix

File: tiago_description/ros2_control/ros2_control.urdf.xacro (robot description, xacro)
@@ -20,19 +20,19 @@
   <xacro:include filename="$(find ${base_type}_description)/urdf/sensors/sensors.ros2_control.xacro"/>
   <xacro:include filename="$(arg description_calibration_dir)/calibration_constants.urdf.xacro" />
+  <xacro:if value="${has_arm}">
+    <xacro:include filename="$(find tiago_description)/urdf/arm/arm.ros2_control.xacro" />
+    <xacro:include filename="$(find tiago_description)/urdf/arm/wrist.ros2_control.xacro" />
+    <xacro:if value="${end_effector == 'pal-gripper'}">
+      <xacro:include filename="$(find pal_gripper_description)/urdf/gripper.ros2_control.xacro" />
+    </xacro:if>
+    <xacro:if value="${end_effector == 'pal-hey5'}">
+      <xacro:include filename="$(find pal_hey5_description)/urdf/pal_hey5.ros2_control.xacro" />
+    </xacro:if>
+    <xacro:if value="${end_effector in ['robotiq-2f-85', 'robotiq-2f-140']}">
+      <xacro:include filename="$(find pal_robotiq_description)/urdf/robotiq.ros2_control.xacro" />
+    </xacro:if>
+  </xacro:if>
   <!-- MACRO DEFINITION-->
   <xacro:macro name="tiago_ros2_control">
-    <xacro:if value="${has_arm}">
-      <xacro:include filename="$(find tiago_description)/urdf/arm/arm.ros2_control.xacro" />
-      <xacro:include filename="$(find tiago_description)/urdf/arm/wrist.ros2_control.xacro" />
-      <xacro:if value="${end_effector == 'pal-gripper'}">
-        <xacro:include filename="$(find pal_gripper_description)/urdf/gripper.ros2_control.xacro" />
-      </xacro:if>
-      <xacro:if value="${end_effector == 'pal-hey5'}">
-        <xacro:include filename="$(find pal_hey5_description)/urdf/pal_hey5.ros2_control.xacro" />
-      </xacro:if>
-      <xacro:if value="${end_effector in ['robotiq-2f-85', 'robotiq-2f-140']}">
-        <xacro:include filename="$(find pal_robotiq_description)/urdf/robotiq.ros2_control.xacro" />
-      </xacro:if>
-    </xacro:if>
     <!-- ROS 2 config-->
     <ros2_control name="ros2_control_tiago_system" type="system">
@@ -63,14 +63,19 @@
       <!-- Torso -->
       <xacro:ros2_control_torso name="torso_lift" reduction="1.0" />
-      <!-- arm -->
+      <!-- Arm -->
       <xacro:if value="${has_arm}">
-        <!-- arm -->
+        <!-- Arm -->
         <xacro:ros2_control_arm name="arm_1" reduction="1.0" offset="${arm_1_joint_offset}" />
         <xacro:ros2_control_arm name="arm_2" reduction="1.0" offset="${arm_2_joint_offset}" />
         <xacro:ros2_control_arm name="arm_3" reduction="1.0" offset="${arm_3_joint_offset}" />
         <xacro:ros2_control_arm name="arm_4" reduction="1.0" offset="${arm_4_joint_offset}" />
-        <!-- wrist -->
+        <!-- Wrist -->
         <xacro:ros2_control_wrist_rotational name="arm_5" reduction="1.0" offset="${arm_5_joint_offset}" />
         <xacro:ros2_control_wrist_differential name="arm" number_1="6" number_2="7" act_reduction_1="-1.0" act_reduction_2="1.0" jnt_reduction_1="1.0" jnt_reduction_2="-1.0" number_1_offset="${arm_6_joint_offset}" number_2_offset="${arm_7_joint_offset}" />
+        <!-- Force Torque sensor -->
+        <xacro:if value="${has_ft_sensor}">
+          <xacro:include filename="$(find tiago_description)/urdf/sensors/sensors.ros2_control.xacro"/>
+          <xacro:ros2_control_force_torque_sensor name="wrist_ft_sensor"/>
+        </xacro:if>
         <!-- End effector -->
         <xacro:if value="${end_effector == 'pal-gripper'}">
@@ -88,9 +93,4 @@
         </xacro:if>
       </xacro:if>
-      <!-- Force Torque sensor -->
-      <xacro:if value="${has_ft_sensor}">
-        <xacro:include filename="$(find tiago_description)/urdf/sensors/sensors.ros2_control.xacro"/>
-        <xacro:ros2_control_force_torque_sensor name="wrist_ft_sensor"/>
-      </xacro:if>
       <!-- Head -->
       <xacro:ros2_control_head name="head_1" reduction="1.0" offset="${head_1_joint_offset}" />

File: tiago_description/urdf/head/head.urdf.xacro (robot description, xacro)
@@ -1,5 +1,5 @@
 <?xml version="1.0"?>
 <!--
-  Copyright (c) 2022 PAL Robotics S.L. All rights reserved.
+  Copyright (c) 2024 PAL Robotics S.L. All rights reserved.
   Licensed under the Apache License, Version 2.0 (the "License");
   you may not use this file except in compliance with the License.
@@ -21,4 +21,5 @@
   <xacro:property name="head_2_lower_limit" value="-60"/>
   <xacro:property name="head_2_upper_limit" value="45"/>
+  <xacro:property name="head_eps" value="${0.00 if no_safety_eps else 0.07}" />
   <!-- INCLUDES -->
   <xacro:include filename="$(find pal_urdf_utils)/urdf/deg_to_rad.urdf.xacro" />
@@ -101,7 +102,4 @@
   <!-- Complete head -->
   <xacro:macro name="head" params="name parent camera_model description_calibration_dir extrinsic_calibration_dir no_safety_eps:=False">
-    <!-- PROPERTIES -->
-    <xacro:property name="head_eps" value="${0.00 if no_safety_eps else 0.07}" />
-    <!-- HEAD DEFINITION -->
     <!-- Head links -->
     <xacro:head_1 name="${name}_1" parent="${parent}" />

File: tiago_description/urdf/torso/torso.ros2_control.xacro (robot description, xacro)
@@ -1,5 +1,5 @@
 <?xml version="1.0"?>
 <!--
-  Copyright (c) 2022 PAL Robotics S.L. All rights reserved.
+  Copyright (c) 2024 PAL Robotics S.L. All rights reserved.
   Licensed under the Apache License, Version 2.0 (the "License");
   you may not use this file except in compliance with the License.
@@ -13,4 +13,7 @@
  -->
 <robot xmlns:xacro="http://ros.org/wiki/xacro">
+  <!-- INCLUDES -->
+  <xacro:include filename="$(find tiago_description)/ros2_control/transmissions.urdf.xacro" />
+  <!-- MACRO DEFINITION-->
   <xacro:macro name="ros2_control_torso" params="name reduction">
     <joint name="${name}_joint">
@@ -20,5 +23,4 @@
       <state_interface name="effort" />
     </joint>
-    <xacro:include filename="$(find tiago_description)/ros2_control/transmissions.urdf.xacro" />
     <xacro:tiago_simple_transmission name="${name}" reduction="${reduction}" />
   </xacro:macro>
