Commit message: Gazebo config std

File: tiago_description/gazebo/gazebo.urdf.xacro (robot description, xacro)
@@ -1,5 +1,5 @@
 <?xml version="1.0"?>
 <!--
-  Copyright (c) 2022 PAL Robotics S.L. All rights reserved.
+  Copyright (c) 2024 PAL Robotics S.L. All rights reserved.
   Licensed under the Apache License, Version 2.0 (the "License");
   you may not use this file except in compliance with the License.
@@ -15,4 +15,5 @@
   xmlns:xacro="http://ros.org/wiki/xacro">
   <gazebo>
+    <!-- ROS2 control plugin -->
     <plugin filename="libgazebo_ros2_control.so" name="gazebo_ros2_control">
       <!-- in the future move this param file somewhere else -->
@@ -25,4 +26,5 @@
       </xacro:unless>
     </plugin>
+    <!-- OMNI BASE PLUGINS -->
     <xacro:if value="${base_type == 'omni_base'}">
       <plugin name="gazebo_ros_planar_move" filename="libgazebo_ros_planar_move.so">
@@ -47,31 +49,16 @@
       </plugin>
     </xacro:if>
-    <plugin filename="libgazebo_ros_p3d.so" name="gazebo_ros_p3d">
-      <body_name>base_footprint</body_name>
-      <always_on>true</always_on>
-      <update_rate>100.0</update_rate>
-      <ros>
-        <remapping>odom:=ground_truth_odom</remapping>
-      </ros>
-      <xacro:if value="${is_multiple}">
-        <!--<robotNamespace>/${nsp}</robotNamespace>-->
-      </xacro:if>
-    </plugin>
+    <!-- PMB2 PLUGINS -->
+    <xacro:if value="${base_type == 'pmb2'}">
+      <plugin filename="libgazebo_world_odometry.so" name="gazebo_ros_odometry">
+        <frame_name>world</frame_name>
+        <body_name>base_footprint</body_name>
+        <topic_name>ground_truth_odom</topic_name>
+        <update_rate>100.0</update_rate>
+        <xacro:if value="${is_multiple}">
+          <namespace>/${nsp}</namespace>
+        </xacro:if>
+      </plugin>
+    </xacro:if>
   </gazebo>
-  <gazebo>
-    <!--- backwards compatibility, used to be gazebo_world_odometry pal plugin-->
-    <plugin filename="libgazebo_ros_p3d.so" name="gazebo_ros_odometry">
-      <body_name>base_footprint</body_name>
-      <always_on>true</always_on>
-      <update_rate>1000.0</update_rate>
-      <ros>
-        <remapping>odom:=floating_base_pose_simulated</remapping>
-      </ros>
-      <xacro:if value="${is_multiple}">
-        <!--<robotNamespace>/${nsp}</robotNamespace>-->
-      </xacro:if>
-    </plugin>
-  </gazebo>
-  <!-- define global properties -->
-  <xacro:property name="M_PI" value="3.1415926535897931" />
 </robot>

File: tiago_description/urdf/sensors/openni.gazebo.xacro (robot description, xacro)
@@ -13,4 +13,6 @@
  -->
 <robot xmlns:xacro="http://ros.org/wiki/xacro">
+  <!-- INCLUDES -->
+  <xacro:include filename="$(find pal_urdf_utils)/urdf/pi.urdf.xacro" />
   <!-- MACRO DEFINITION-->
   <xacro:macro name="openni_camera_gazebo_v0" params="name">
