Commit message: Add base_type parameter

File: tiago_description/robots/tiago.urdf.xacro (robot description, xacro)
@@ -26,4 +26,5 @@
     <xacro:arg name="namespace" default=""/>
     <xacro:arg name="no_safety_eps" default="false"/>
+    <xacro:arg name="base_type" default="pmb2"/> <!-- pmb2, omni_base -->
     <xacro:arg name="use_sim" default="false"/>
     <xacro:property name="arm" value="$(arg arm)" />
@@ -38,4 +39,5 @@
     <xacro:property name="is_multiple" value="$(arg multiple)" />
     <xacro:property name="nsp" value="$(arg namespace)" />
+    <xacro:property name="base_type" value="$(arg base_type)" />
     <xacro:property name="no_safety_eps" value="$(arg no_safety_eps)" />
     <xacro:property name="has_arm" value="${arm != 'no-arm'}"/>
@@ -57,4 +59,7 @@
     <xacro:wrong_camera_model/>
   </xacro:if>
+  <xacro:if value="${base_type not in ['pmb2', 'omni_base']}">
+    <xacro:wrong_base_type/>
+  </xacro:if>
         <!-- The properties below are modified using empy http://www.alcyone.com/software/empy/
              from the create_robot.py tool. Handle them with care -->
@@ -67,5 +72,5 @@
   <!-- The following included files set up definitions of parts of the robot body -->
   <!-- Base -->
-  <xacro:include filename="$(find pmb2_description)/urdf/base/base_sensors.urdf.xacro" />
+  <xacro:include filename="$(find ${base_type}_description)/urdf/base/base_sensors.urdf.xacro" />
   <!-- Torso -->
   <xacro:include filename="$(find tiago_description)/urdf/torso/torso.urdf.xacro" />
@@ -92,5 +97,10 @@
   <xacro:include filename="$(find pal_urdf_utils)/urdf/materials.urdf.xacro" />
   <!-- Now we can start using the macros included above to define the actual robot -->
-  <xacro:base_sensors name="base" laser_model="$(arg laser_model)" sonars="true" microphone="true"/>
+  <xacro:if value="${base_type == 'pmb2'}">
+    <xacro:base_sensors name="base" laser_model="$(arg laser_model)" sonars="true" microphone="true"/>
+  </xacro:if>
+  <xacro:if value="${base_type == 'omni_base'}">
+    <xacro:base_sensors name="base" front_laser_model="$(arg laser_model)" rear_laser_model="$(arg laser_model)"/>
+  </xacro:if>
   <xacro:tiago_torso name="torso" parent="base_link"/>
   <xacro:head name="head" parent="torso_lift_link" camera_model="$(arg camera_model)"

Commit message: High level urdf standarization

File: tiago_description/robots/tiago.urdf.xacro (robot description, xacro)
@@ -1,5 +1,5 @@
 <?xml version="1.0"?>
 <!--
-  Copyright (c) 2022 PAL Robotics S.L. All rights reserved.
+  Copyright (c) 2024 PAL Robotics S.L. All rights reserved.
   Licensed under the Apache License, Version 2.0 (the "License");
   you may not use this file except in compliance with the License.
@@ -12,38 +12,50 @@
   limitations under the License.
  -->
-<robot  xmlns:xacro="http://ros.org/wiki/xacro"
-        name="tiago" >
-    <xacro:arg name="arm" default="tiago-arm"/> <!-- tiago-arm, no-arm -->
-    <xacro:arg name="wrist_model" default="wrist-2010"/>
-    <xacro:arg name="end_effector" default="pal-hey5"/> <!-- no-end-effector, pal-gripper, pal-hey5-->
-    <xacro:arg name="ft_sensor" default="schunk-ft"/> <!-- no-ft-sensor, schunk-ft -->
-    <xacro:arg name="laser_model" default="sick-571"/> <!-- no-laser, hokuyo, sick-551, sick-561, sick-571-->
-    <xacro:arg name="camera_model" default="orbbec-astra"/> <!-- no-camera, orbbec-astra, orbbec-astra-pro, asus-xtion -->
-    <xacro:arg name="has_thermal_camera" default="false"/>
-    <xacro:arg name="multiple" default="false"/>
-    <xacro:arg name="description_calibration_dir" default="$(find tiago_description)/urdf/calibration"/>
-    <xacro:arg name="extrinsic_calibration_dir" default="$(find tiago_description)/urdf/calibration"/>
-    <xacro:arg name="namespace" default=""/>
-    <xacro:arg name="no_safety_eps" default="false"/>
-    <xacro:arg name="base_type" default="pmb2"/> <!-- pmb2, omni_base -->
-    <xacro:arg name="use_sim" default="false"/>
-    <xacro:property name="arm" value="$(arg arm)" />
-    <xacro:if value="${arm not in ['tiago-arm', 'no-arm']}">
-      <xacro:wrong_arm/>
-    </xacro:if>
-    <xacro:property name="wrist_model" value="$(arg wrist_model)" />
-    <xacro:property name="end_effector" value="$(arg end_effector)" />
-    <xacro:property name="ft_sensor" value="$(arg ft_sensor)" />
-    <xacro:property name="laser_model" value="$(arg laser_model)" />
-    <xacro:property name="camera_model" value="$(arg camera_model)" />
-    <xacro:property name="is_multiple" value="$(arg multiple)" />
-    <xacro:property name="nsp" value="$(arg namespace)" />
-    <xacro:property name="base_type" value="$(arg base_type)" />
-    <xacro:property name="no_safety_eps" value="$(arg no_safety_eps)" />
-    <xacro:property name="has_arm" value="${arm != 'no-arm'}"/>
-  <xacro:if value="${has_arm}">
-    <xacro:if value="${wrist_model not in ['wrist-2010', 'wrist-2017']}">
-      <xacro:wrong_wrist_model/>
-    </xacro:if>
+<robot xmlns:xacro="http://ros.org/wiki/xacro" name="tiago">
+  <!-- ARGUMENTS -->
+  <!-- no-arm, tiago-arm -->
+  <xacro:arg name="arm_model" default="tiago-arm"/>
+  <!-- no-end-effector, pal-gripper, pal-hey5-->
+  <xacro:arg name="end_effector" default="pal-hey5"/>
+  <!-- no-ft-sensor, schunk-ft -->
+  <xacro:arg name="ft_sensor" default="schunk-ft"/>
+  <!-- no-laser, hokuyo, sick-551, sick-561, sick-571-->
+  <xacro:arg name="laser_model" default="sick-571"/>
+  <!-- no-camera, orbbec-astra, orbbec-astra-pro, asus-xtion -->
+  <xacro:arg name="camera_model" default="orbbec-astra"/>
+  <!-- pmb2, omni_base -->
+  <xacro:arg name="base_type" default="pmb2"/>
+  <xacro:arg name="use_sim" default="false"/>
+  <xacro:arg name="has_thermal_camera" default="false"/>
+  <xacro:arg name="multiple" default="false"/>
+  <xacro:arg name="description_calibration_dir" default="$(find tiago_description)/urdf/calibration"/>
+  <xacro:arg name="extrinsic_calibration_dir" default="$(find tiago_description)/urdf/calibration"/>
+  <xacro:arg name="namespace" default=""/>
+  <xacro:arg name="no_safety_eps" default="false"/>
+  <xacro:arg name="wrist_model" default="wrist-2010"/>
+  <!-- PROPERTIES -->
+  <xacro:property name="wrist_model" value="$(arg wrist_model)" />
+  <xacro:property name="end_effector" value="$(arg end_effector)" />
+  <xacro:property name="ft_sensor" value="$(arg ft_sensor)" />
+  <xacro:property name="laser_model" value="$(arg laser_model)" />
+  <xacro:property name="camera_model" value="$(arg camera_model)" />
+  <xacro:property name="is_multiple" value="$(arg multiple)" />
+  <xacro:property name="nsp" value="$(arg namespace)" />
+  <xacro:property name="base_type" value="$(arg base_type)" />
+  <xacro:property name="no_safety_eps" value="$(arg no_safety_eps)" />
+  <xacro:property name="arm_model" value="$(arg arm_model)" />
+  <xacro:property name="has_arm" value="${arm_model not in ['no-arm']}"/>
+  <xacro:property name="has_ft_sensor" value="${ft_sensor not in ['no-ft-sensor'] and has_arm}"/>
+  <xacro:property name="has_end_effector" value="${end_effector not in ['no-end-effector']}"/>
+  <xacro:property name="end_effector_link" value="${'wrist_ft_tool_link' if has_ft_sensor else 'arm_tool_link'}"/>
+  <xacro:property name="end_effector_name" value="${'hand' if end_effector == 'pal-hey5' else 'gripper'}"/>
+  <xacro:property name="head_link_name" value="head_2_link"/>
+  <xacro:property name="description_calibration_dir" value="${arg description_calibration_dir}"/>
+  <!-- Properties check -->
+  <xacro:if value="${arm_model not in ['tiago-arm', 'no-arm']}">
+    <xacro:wrong_arm/>
+  </xacro:if>
+  <xacro:if value="${wrist_model not in ['wrist-2010', 'wrist-2017']}">
+    <xacro:wrong_wrist_model/>
   </xacro:if>
   <xacro:if value="${end_effector not in ['no-end-effector', 'pal-gripper', 'pal-hey5', 'custom', 'robotiq-2f-85', 'robotiq-2f-140']}">
@@ -62,22 +74,20 @@
     <xacro:wrong_base_type/>
   </xacro:if>
-        <!-- The properties below are modified using empy http://www.alcyone.com/software/empy/
-             from the create_robot.py tool. Handle them with care -->
-   <xacro:property name="has_schunk_ft"           value="${ft_sensor == 'schunk-ft'}"/>
-   <xacro:property name="has_ft_sensor"           value="${has_arm and has_schunk_ft}"/> <!-- This should be OR'ed with other FT sensors-->
-   <xacro:property name="end_effector_link"       value="${'wrist_ft_tool_link' if has_ft_sensor else 'arm_tool_link'}"/>
-   <xacro:property name="end_effector_name"       value="${'hand' if end_effector == 'pal-hey5' else 'gripper'}"/>
-   <xacro:property name="head_link_name"          value="head_2_link"/>
-   <xacro:property name="description_calibration_dir"       value="${arg description_calibration_dir}"/>
-  <!-- The following included files set up definitions of parts of the robot body -->
+  <!-- INCLUDES -->
+  <!-- Tools -->
+  <xacro:include filename="$(find pal_urdf_utils)/urdf/deg_to_rad.urdf.xacro" />
   <!-- Base -->
   <xacro:include filename="$(find ${base_type}_description)/urdf/base/base_sensors.urdf.xacro" />
   <!-- Torso -->
   <xacro:include filename="$(find tiago_description)/urdf/torso/torso.urdf.xacro" />
+  <!-- Calibration constants -->
+  <xacro:include filename="$(arg description_calibration_dir)/calibration_constants.urdf.xacro" />
+  <!-- Arm -->
   <xacro:if value="${has_arm}">
-    <!-- Arm -->
     <xacro:include filename="$(find tiago_description)/urdf/arm/arm.urdf.xacro" />
+  </xacro:if>
+  <!-- End effector -->
+  <xacro:if value="${has_arm and has_end_effector}">
     <xacro:include filename="$(find tiago_description)/urdf/end_effector/end_effector.urdf.xacro" />
-    <xacro:include filename="$(arg description_calibration_dir)/calibration_constants.urdf.xacro" />
   </xacro:if>
   <!-- Force Torque sensor -->
@@ -88,13 +98,12 @@
   <!-- Head -->
   <xacro:include filename="$(find tiago_description)/urdf/head/head.urdf.xacro" />
+  <!-- Materials for visualization -->
+  <xacro:include filename="$(find pal_urdf_utils)/urdf/materials.urdf.xacro" />
   <!-- Generic simulator_gazebo plugins -->
   <xacro:include filename="$(find tiago_description)/gazebo/gazebo.urdf.xacro" />
-  <!-- ros2_control -->
+  <!-- ROS 2 control -->
   <xacro:include filename="$(find tiago_description)/ros2_control/ros2_control.urdf.xacro" />
-  <xacro:tiago_ros2_control
-    use_sim="$(arg use_sim)" />
-  <!-- Materials for visualization -->
-  <xacro:include filename="$(find pal_urdf_utils)/urdf/materials.urdf.xacro" />
-  <!-- Now we can start using the macros included above to define the actual robot -->
+  <!-- ROBOT DEFINITION -->
+  <!-- Base -->
   <xacro:if value="${base_type == 'pmb2'}">
     <xacro:base_sensors name="base" laser_model="$(arg laser_model)" sonars="true" microphone="true"/>
@@ -103,47 +112,53 @@
     <xacro:base_sensors name="base" front_laser_model="$(arg laser_model)" rear_laser_model="$(arg laser_model)"/>
   </xacro:if>
+  <!-- Torso -->
   <xacro:tiago_torso name="torso" parent="base_link"/>
-  <xacro:head name="head" parent="torso_lift_link" camera_model="$(arg camera_model)"
-	  description_calibration_dir="$(arg description_calibration_dir)"
-	  extrinsic_calibration_dir="$(arg extrinsic_calibration_dir)"
-    no_safety_eps="${no_safety_eps}"/>
+  <!-- Head -->
+  <xacro:head name="head" parent="torso_lift_link" camera_model="$(arg camera_model)" description_calibration_dir="$(arg description_calibration_dir)" extrinsic_calibration_dir="$(arg extrinsic_calibration_dir)" no_safety_eps="${no_safety_eps}"/>
+  <!-- Arm -->
   <xacro:if value="${has_arm}">
-	  <xacro:tiago_arm name="arm" parent="torso_lift_link" wrist_model="${wrist_model}" has_ft_sensor="${has_ft_sensor}" reflect="1" tiago_dual="-1" arm_1_offset="${arm_1_joint_offset}" arm_2_offset="${arm_2_joint_offset}" arm_3_offset="${arm_3_joint_offset}" arm_4_offset="${arm_4_joint_offset}" arm_5_offset="${arm_5_joint_offset}" arm_6_offset="${arm_6_joint_offset}" arm_7_offset="${arm_7_joint_offset}" no_safety_eps="${no_safety_eps}">
-        <origin xyz="0.15505 0.014 -0.151" rpy="0 0 ${-90 * deg_to_rad}" />
-      </xacro:tiago_arm>
+    <!-- Arm -->
+    <xacro:tiago_arm name="arm" parent="torso_lift_link" wrist_model="${wrist_model}" has_ft_sensor="${has_ft_sensor}" reflect="1" tiago_dual="-1" arm_1_offset="${arm_1_joint_offset}" arm_2_offset="${arm_2_joint_offset}" arm_3_offset="${arm_3_joint_offset}" arm_4_offset="${arm_4_joint_offset}" arm_5_offset="${arm_5_joint_offset}" arm_6_offset="${arm_6_joint_offset}" arm_7_offset="${arm_7_joint_offset}" no_safety_eps="${no_safety_eps}">
+      <origin xyz="0.15505 0.014 -0.151" rpy="0 0 ${-90 * deg_to_rad}" />
+    </xacro:tiago_arm>
+    <!-- End effector -->
+    <xacro:if value="${has_end_effector}">
       <xacro:tiago_end_effector name="${end_effector_name}" parent="${end_effector_link}" type="${end_effector}" reflect="1"/>
-  </xacro:if>
-  <!-- Force Torque sensor -->
-  <xacro:if value="${has_ft_sensor}">
+    </xacro:if>
+    <!-- FT sensor -->
+    <xacro:if value="${has_ft_sensor}">
       <xacro:ft_sensor name="wrist" parent="arm_tool_link" />
       <xacro:force_torque_sensor_gazebo name="wrist_ft" update_rate="100"/>
+    </xacro:if>
   </xacro:if>
   <!-- Thermal camera -->
   <xacro:if value="$(arg has_thermal_camera)">
     <joint name="thermal_camera_joint" type="fixed">
-        <parent link="${head_link_name}"/>
-        <child link="thermal_camera"/>
-        <origin xyz="0.05 0.15 0" rpy="${0*deg_to_rad} ${-90*deg_to_rad} ${-180*deg_to_rad}" />
+      <parent link="${head_link_name}"/>
+      <child link="thermal_camera"/>
+      <origin xyz="0.05 0.15 0" rpy="${0*deg_to_rad} ${-90*deg_to_rad} ${-180*deg_to_rad}" />
     </joint>
     <link name="thermal_camera">
-        <inertial>
-            <origin xyz="0 0 0" rpy="0 0 0"/>
-            <mass value="0.0001" />
-            <inertia ixx="0.0001"  ixy="0"  ixz="0" iyy="0.0001" iyz="0" izz="0.0001" />
-        </inertial>
+      <inertial>
+        <origin xyz="0 0 0" rpy="0 0 0"/>
+        <mass value="0.0001" />
+        <inertia ixx="0.0001" ixy="0" ixz="0" iyy="0.0001" iyz="0" izz="0.0001" />
+      </inertial>
     </link>
   </xacro:if>
   <!-- RGBD Laser Link -->
   <joint name="rgbd_laser_joint" type="fixed">
-      <parent link="base_footprint"/>
-      <child link="rgbd_laser_link"/>
-      <origin xyz="-0.9 0 0" rpy="0 0 0" />
+    <parent link="base_footprint"/>
+    <child link="rgbd_laser_link"/>
+    <origin xyz="-0.9 0 0" rpy="0 0 0" />
   </joint>
   <link name="rgbd_laser_link">
-      <inertial>
-          <origin xyz="0 0 0" rpy="0 0 0"/>
-          <mass value="0.0001" />
-          <inertia ixx="0.0001"  ixy="0"  ixz="0" iyy="0.0001" iyz="0" izz="0.0001" />
-      </inertial>
+    <inertial>
+      <origin xyz="0 0 0" rpy="0 0 0"/>
+      <mass value="0.0001" />
+      <inertia ixx="0.0001" ixy="0" ixz="0" iyy="0.0001" iyz="0" izz="0.0001" />
+    </inertial>
   </link>
+  <!-- ROS 2 Control -->
+  <xacro:tiago_ros2_control use_sim="$(arg use_sim)" />
 </robot>

File: tiago_description/ros2_control/ros2_control.urdf.xacro (robot description, xacro)
@@ -1,5 +1,5 @@
 <?xml version="1.0"?>
 <!--
-  Copyright (c) 2022 PAL Robotics S.L. All rights reserved.
+  Copyright (c) 2024 PAL Robotics S.L. All rights reserved.
   Licensed under the Apache License, Version 2.0 (the "License");
   you may not use this file except in compliance with the License.
@@ -12,15 +12,18 @@
   limitations under the License.
  -->
-<robot xmlns:xacro="http://ros.org/wiki/xacro"
-       name="tiago" >
+<robot xmlns:xacro="http://ros.org/wiki/xacro" name="tiago">
   <xacro:macro name="tiago_ros2_control" params="use_sim:=^|false">
-    <xacro:arg name="arm" default="true" />
+    <xacro:arg name="arm_model" default="tiago-arm" />
     <xacro:arg name="end_effector" default="pal-hey5"/>
     <xacro:arg name="description_calibration_dir" default="$(find tiago_description)/urdf/calibration" />
-    <xacro:property name="has_arm" value="${arm != 'no-arm'}" />
-    <xacro:property name="end_effector" value="$(arg end_effector)" />
+    <xacro:property name="has_arm" value="${arm_model not in ['no-arm']}"/>
+    <xacro:property name="has_ft_sensor" value="${ft_sensor not in ['no-ft-sensor'] and has_arm}"/>
+    <xacro:property name="has_end_effector" value="${end_effector not in ['no-end-effector'] and has_arm}"/>
+    <xacro:property name="has_ft_sensor" value="${ft_sensor not in ['no-ft-sensor'] and has_arm}"/>
     <xacro:include filename="$(find ${base_type}_description)/urdf/wheels/wheel.ros2_control.xacro" />
     <xacro:include filename="$(find tiago_description)/urdf/torso/torso.ros2_control.xacro" />
     <xacro:include filename="$(find tiago_description)/urdf/head/head.ros2_control.xacro" />
+    <xacro:include filename="$(find ${base_type}_description)/urdf/sensors/sensors.ros2_control.xacro"/>
+    <xacro:include filename="$(arg description_calibration_dir)/calibration_constants.urdf.xacro" />
     <xacro:if value="${has_arm}">
       <xacro:include filename="$(find tiago_description)/urdf/arm/arm.ros2_control.xacro" />
@@ -36,7 +39,4 @@
       </xacro:if>
     </xacro:if>
-    <xacro:include filename="$(find ${base_type}_description)/urdf/sensors/sensors.ros2_control.xacro"/>
-    <!-- calibration offsets -->
-    <xacro:include filename="$(arg description_calibration_dir)/calibration_constants.urdf.xacro" />
     <ros2_control name="ros2_control_tiago_system" type="system">
       <hardware>
@@ -54,8 +54,8 @@
       </xacro:if>
       <xacro:if value="${base_type == 'omni_base'}">
-	<xacro:ros2_control_wheel side="front_right" />
-	<xacro:ros2_control_wheel side="front_left" />
-	<xacro:ros2_control_wheel side="rear_right" />
-	<xacro:ros2_control_wheel side="rear_left" />
+        <xacro:ros2_control_wheel side="front_right" />
+        <xacro:ros2_control_wheel side="front_left" />
+        <xacro:ros2_control_wheel side="rear_right" />
+        <xacro:ros2_control_wheel side="rear_left" />
       </xacro:if>
       <!-- IMU -->
@@ -76,8 +76,6 @@
         <!-- wrist -->
         <xacro:ros2_control_wrist_rotational name="arm_5" reduction="1.0" offset="${arm_5_joint_offset}" />
-        <xacro:ros2_control_wrist_differential name="arm" number_1="6" number_2="7"
-                                               act_reduction_1="-1.0" act_reduction_2="1.0"
-                                               jnt_reduction_1="1.0" jnt_reduction_2="-1.0"
-                                               number_1_offset="${arm_6_joint_offset}" number_2_offset="${arm_7_joint_offset}" />
+        <xacro:ros2_control_wrist_differential name="arm" number_1="6" number_2="7" act_reduction_1="-1.0" act_reduction_2="1.0" jnt_reduction_1="1.0" jnt_reduction_2="-1.0" number_1_offset="${arm_6_joint_offset}" number_2_offset="${arm_7_joint_offset}" />
+        <!-- End effector -->
         <xacro:if value="${end_effector == 'pal-gripper'}">
           <!-- pal-gripper -->

File: tiago_description/ros2_control/transmissions.urdf.xacro (robot description, xacro)
@@ -13,20 +13,19 @@
  -->
 <robot xmlns:xacro="http://ros.org/wiki/xacro">
-  <xacro:macro name="tiago_simple_transmission" params="name reduction:=1.0 offset_value:=0.0" >
+  <xacro:macro name="tiago_simple_transmission" params="name reduction:=1.0 offset_value:=0.0">
     <transmission name="${name}_trans">
       <plugin>transmission_interface/SimpleTransmission</plugin>
-      <actuator name="${name}_actuator"  role="actuator1"/>
+      <actuator name="${name}_actuator" role="actuator1"/>
       <joint name="${name}_joint" role="joint1">
         <mechanical_reduction>${reduction}</mechanical_reduction>
         <offset>${offset_value}</offset>
-     </joint>
+      </joint>
     </transmission>
   </xacro:macro>
-  <xacro:macro name="tiago_differential_transmission"
-               params="name number_1 number_2 act_reduction_1 act_reduction_2 jnt_reduction_1 jnt_reduction_2 number_1_offset number_2_offset" >
-  <transmission name="${name}_${number_1}_${name}_${number_2}_wrist_trans">
+  <xacro:macro name="tiago_differential_transmission" params="name number_1 number_2 act_reduction_1 act_reduction_2 jnt_reduction_1 jnt_reduction_2 number_1_offset number_2_offset">
+    <transmission name="${name}_${number_1}_${name}_${number_2}_wrist_trans">
       <plugin>transmission_interface/DifferentialTransmission</plugin>
       <actuator name="${name}_${number_1}_actuator" role="actuator1">
-      <mechanical_reduction>${act_reduction_1}</mechanical_reduction>
+        <mechanical_reduction>${act_reduction_1}</mechanical_reduction>
       </actuator>
       <actuator name="${name}_${number_2}_actuator" role="actuator2">
