Commit message: Head std

File: tiago_description/robots/tiago.urdf.xacro (robot description, xacro)
@@ -37,4 +37,6 @@
   <!-- no-camera, orbbec-astra, orbbec-astra-pro, asus-xtion -->
   <xacro:arg name="camera_model" default="orbbec-astra"/>
+  <!-- false, true -->
+  <xacro:arg name="has_thermal_camera" default="false"/>
   <!-- false, true -->
   <xacro:arg name="no_safety_eps" default="false"/>
@@ -85,4 +87,5 @@
   <xacro:property name="end_effector_link" value="${'wrist_ft_tool_link' if has_ft_sensor else 'arm_tool_link'}"/>
   <xacro:property name="end_effector_name" value="${'hand' if end_effector == 'pal-hey5' else 'gripper'}"/>
+  <xacro:property name="has_thermal_camera" default="$(arg has_thermal_camera)"/>
   <xacro:property name="arm_x" default="0.08976" />
   <xacro:property name="arm_y" default="0.15918" />
@@ -92,6 +95,6 @@
   <xacro:property name="arm_yaw" default="-1.2217" />
   <!-- Calibration -->
-  <xacro:property name="description_calibration_dir" value="${arg description_calibration_dir}"/>
-  <xacro:property name="extrinsic_calibration_dir" value="${arg extrinsic_calibration_dir}"/>
+  <xacro:property name="description_calibration_dir" value="$(arg description_calibration_dir)"/>
+  <xacro:property name="extrinsic_calibration_dir" value="$(arg extrinsic_calibration_dir)"/>
   <!-- Execution env configuration -->
   <xacro:property name="use_sim_time" default="$(arg is_multiple)"/>
@@ -121,5 +124,5 @@
   <xacro:include filename="$(find pal_urdf_utils)/urdf/deg_to_rad.urdf.xacro" />
   <!-- Calibration constants -->
-  <xacro:include filename="$(arg description_calibration_dir)/calibration_constants.urdf.xacro" />
+  <xacro:include filename="${description_calibration_dir}/calibration_constants.urdf.xacro" />
   <!-- Materials for visualization -->
   <xacro:include filename="$(find pal_urdf_utils)/urdf/materials.urdf.xacro" />
@@ -139,5 +142,5 @@
   <xacro:tiago_torso name="torso" parent="base_link"/>
   <!-- Head -->
-  <xacro:head name="head" parent="torso_lift_link" camera_model="${camera_model}" description_calibration_dir="${description_calibration_dir}" extrinsic_calibration_dir="$(arg extrinsic_calibration_dir)" no_safety_eps="${no_safety_eps}"/>
+  <xacro:head name="head" parent="torso_lift_link" camera_model="${camera_model}" description_calibration_dir="${description_calibration_dir}" extrinsic_calibration_dir="${extrinsic_calibration_dir}" no_safety_eps="${no_safety_eps}"/>
   <!-- Arm -->
   <xacro:if value="${has_arm}">

File: tiago_description/urdf/head/head.urdf.xacro (robot description, xacro)
@@ -13,19 +13,18 @@
  -->
 <robot xmlns:xacro="http://ros.org/wiki/xacro">
-  <!--File includes-->
-  <xacro:include filename="$(find pal_urdf_utils)/urdf/deg_to_rad.urdf.xacro" />
-  <xacro:include filename="$(find tiago_description)/urdf/sensors/xtion_pro_live.urdf.xacro" />
-  <xacro:include filename="$(find tiago_description)/urdf/sensors/orbbec_astra.urdf.xacro" />
-  <!--Constant parameters-->
+  <!-- PROPERTIES -->
   <xacro:property name="head_friction" value="1.0" />
-  <xacro:property name="head_damping"  value="0.5" />
-  <xacro:property name="head_max_vel"  value="3.0" />
+  <xacro:property name="head_damping" value="0.5" />
+  <xacro:property name="head_max_vel" value="3.0" />
   <xacro:property name="head_1_lower_limit" value="-75"/>
   <xacro:property name="head_1_upper_limit" value="75"/>
   <xacro:property name="head_2_lower_limit" value="-60"/>
   <xacro:property name="head_2_upper_limit" value="45"/>
-  <!--************************-->
-  <!--     HEAD_1 (PAN)       -->
-  <!--************************-->
+  <!-- INCLUDES -->
+  <xacro:include filename="$(find pal_urdf_utils)/urdf/deg_to_rad.urdf.xacro" />
+  <xacro:include filename="$(find tiago_description)/urdf/sensors/xtion_pro_live.urdf.xacro" />
+  <xacro:include filename="$(find tiago_description)/urdf/sensors/orbbec_astra.urdf.xacro" />
+  <!-- MACRO DEFINITION-->
+  <!-- head_1 (pan) -->
   <xacro:macro name="head_1" params="name parent">
     <link name="${name}_link">
@@ -33,7 +32,5 @@
         <origin xyz="-0.00508 0.00237 0.07229" rpy="0.00000 0.00000 0.00000"/>
         <mass value="0.62220"/>
-        <inertia ixx="0.00119200000" ixy="-0.00000700000" ixz="0.00009600000"
-                 iyy="0.00140200000" iyz="0.00000400000"
-                 izz="0.00088900000"/>
+        <inertia ixx="0.00119200000" ixy="-0.00000700000" ixz="0.00009600000" iyy="0.00140200000" iyz="0.00000400000" izz="0.00088900000"/>
       </inertial>
       <visual>
@@ -55,12 +52,9 @@
       <parent link="${parent}"/>
       <child link="${name}_link"/>
-      <origin xyz="0.182 0.0 0.0"  rpy="0 0 0" />
+      <origin xyz="0.182 0.0 0.0" rpy="0 0 0" />
       <axis xyz="0 0 1" />
       <limit lower="${head_1_lower_limit * deg_to_rad}" upper="${head_1_upper_limit * deg_to_rad}" effort="5.197" velocity="${head_max_vel}" />
       <dynamics damping="${head_damping}" friction="${head_friction}"/>
-      <safety_controller k_position="20"
-                         k_velocity="20"
-                         soft_lower_limit="${head_1_lower_limit * deg_to_rad + head_eps}"
-                         soft_upper_limit="${head_1_upper_limit * deg_to_rad - head_eps}" />
+      <safety_controller k_position="20" k_velocity="20" soft_lower_limit="${head_1_lower_limit * deg_to_rad + head_eps}" soft_upper_limit="${head_1_upper_limit * deg_to_rad - head_eps}" />
     </joint>
     <gazebo reference="${name}_link">
@@ -69,10 +63,8 @@
     </gazebo>
     <gazebo reference="${name}_joint">
-       <implicitSpringDamper>1</implicitSpringDamper>
+      <implicitSpringDamper>1</implicitSpringDamper>
     </gazebo>
   </xacro:macro>
-  <!--************************-->
-  <!--      HEAD_2 (TILT)     -->
-  <!--************************-->
+  <!-- head_2 (tilt) -->
   <xacro:macro name="head_2" params="name parent">
     <link name="${name}_link">
@@ -80,7 +72,5 @@
         <origin xyz="0.04700 0.05542 0.00022" rpy="0.00000 0.00000 0.00000"/>
         <mass value="0.66123"/>
-        <inertia ixx="0.00462000000" ixy="0.00068900000" ixz="0.00000600000"
-                 iyy="0.00486100000" iyz="0.00000600000"
-                 izz="0.00313200000"/>
+        <inertia ixx="0.00462000000" ixy="0.00068900000" ixz="0.00000600000" iyy="0.00486100000" iyz="0.00000600000" izz="0.00313200000"/>
       </inertial>
       <visual>
@@ -101,20 +91,23 @@
       <parent link="${parent}"/>
       <child link="${name}_link"/>
-      <origin xyz="0.005 0.0 0.098"  rpy="${90.0 * deg_to_rad} 0 0" />
+      <origin xyz="0.005 0.0 0.098" rpy="${90.0 * deg_to_rad} 0 0" />
       <axis xyz="0 0 1" />
       <limit lower="${head_2_lower_limit * deg_to_rad}" upper="${head_2_upper_limit * deg_to_rad}" effort="2.77" velocity="${head_max_vel}" />
       <dynamics damping="${head_damping}" friction="${head_friction}"/>
-      <safety_controller k_position="20"
-                         k_velocity="20"
-                         soft_lower_limit="${head_2_lower_limit * deg_to_rad + head_eps}"
-                         soft_upper_limit="${head_2_upper_limit * deg_to_rad - head_eps}" />
+      <safety_controller k_position="20" k_velocity="20" soft_lower_limit="${head_2_lower_limit * deg_to_rad + head_eps}" soft_upper_limit="${head_2_upper_limit * deg_to_rad - head_eps}" />
     </joint>
   </xacro:macro>
+  <!-- Complete head -->
   <xacro:macro name="head" params="name parent camera_model description_calibration_dir extrinsic_calibration_dir no_safety_eps:=False">
-    <xacro:property name="head_eps"      value="${0.00 if no_safety_eps else 0.07}" />
-    <!-- includes -->
+    <!-- PROPERTIES -->
+    <xacro:property name="head_eps" value="${0.00 if no_safety_eps else 0.07}" />
+    <!-- INCLUDES -->
     <xacro:include filename="$(arg description_calibration_dir)/calibration_constants.urdf.xacro" />
+    <!-- HEAD DEFINITION -->
+    <!-- Head links -->
     <xacro:head_1 name="${name}_1" parent="${parent}" />
     <xacro:head_2 name="${name}_2" parent="${name}_1_link"/>
+    <!-- Cameras-->
+    <!-- Asus Xtion-->
     <xacro:if value="${camera_model == 'asus-xtion'}">
       <xacro:xtion_pro_live name="head_front_camera" parent="${name}_2" camera_model="${camera_model}" extrinsic_calibration_dir="${extrinsic_calibration_dir}">
@@ -124,4 +117,5 @@
       </xacro:xtion_pro_live>
     </xacro:if>
+    <!-- Orbecc Astra-->
     <xacro:if value="${camera_model in ['orbbec-astra', 'orbbec-astra-pro']}">
       <xacro:orbbec_astra name="head_front_camera" parent="${name}_2" camera_model="${camera_model}" extrinsic_calibration_dir="${extrinsic_calibration_dir}">

File: tiago_description/urdf/sensors/openni.gazebo.xacro (robot description, xacro)
@@ -13,4 +13,5 @@
  -->
 <robot xmlns:xacro="http://ros.org/wiki/xacro">
+  <!-- MACRO DEFINITION-->
   <xacro:macro name="openni_camera_gazebo_v0" params="name">
     <gazebo reference="${name}_rgb_frame">
@@ -29,5 +30,5 @@
             <far>8.0</far>
           </clip>
-	  <distortion>
+          <distortion>
             <k1>0.00000001</k1>
             <k2>0.00000001</k2>
@@ -40,10 +41,10 @@
           <camera_name>${name}</camera_name>
           <ros>
-			  <!-- <namespace>${name}</namespace>-->
-	    <remapping>${name}/image_raw:=${name}/rgb/image_raw</remapping>
-	    <remapping>${name}/camera_info:=${name}/rgb/camera_info</remapping>
-	    <remapping>${name}/depth/image_raw:=${name}/depth_registered/image_raw</remapping>
-	    <remapping>${name}/depth/camera_info:=${name}/depth_registered/camera_info</remapping>
-	    <remapping>${name}/points:=${name}/depth_registered/points</remapping>
+            <!-- <namespace>${name}</namespace>-->
+            <remapping>${name}/image_raw:=${name}/rgb/image_raw</remapping>
+            <remapping>${name}/camera_info:=${name}/rgb/camera_info</remapping>
+            <remapping>${name}/depth/image_raw:=${name}/depth_registered/image_raw</remapping>
+            <remapping>${name}/depth/camera_info:=${name}/depth_registered/camera_info</remapping>
+            <remapping>${name}/points:=${name}/depth_registered/points</remapping>
           </ros>
           <frame_name>${name}_rgb_optical_frame</frame_name>

File: tiago_description/urdf/sensors/orbbec_astra.urdf.xacro (robot description, xacro)
@@ -1,5 +1,5 @@
 <?xml version="1.0"?>
 <!--
-  Copyright (c) 2022 PAL Robotics S.L. All rights reserved.
+  Copyright (c) 2024 PAL Robotics S.L. All rights reserved.
   Licensed under the Apache License, Version 2.0 (the "License");
   you may not use this file except in compliance with the License.
@@ -14,8 +14,9 @@
 <!--  Orbbec Astra based off ASUS Xtion Pro Live-->
 <robot xmlns:xacro="http://ros.org/wiki/xacro">
+  <!-- INCLUDES -->
   <xacro:include filename="$(find tiago_description)/urdf/sensors/openni.gazebo.xacro" />
-  <!-- Macro -->
+  <!-- MACRO DEFINITION-->
   <xacro:macro name="orbbec_astra" params="name parent camera_model *origin *optical_origin extrinsic_calibration_dir">
-    <!-- includes -->
+    <!-- INCLUDES -->
     <xacro:include filename="${extrinsic_calibration_dir}/extrinsic_camera_calibration_constants.urdf.xacro" />
     <!-- frames in the center of the camera -->
@@ -29,7 +30,5 @@
         <origin xyz="-0.00936000000 -0.00003000000 -0.00273000000" rpy="0 0 0"/>
         <mass value="0.21970000000"/>
-        <inertia ixx="0.00000429247" ixy="0.00000000000" ixz="0.00000002565"
-                 iyy="0.00000008027" iyz="0.00000000000"
-                 izz="0.00000427339"/>
+        <inertia ixx="0.00000429247" ixy="0.00000000000" ixz="0.00000002565" iyy="0.00000008027" iyz="0.00000000000" izz="0.00000427339"/>
       </inertial>
       <!--
@@ -60,7 +59,5 @@
         <origin xyz="0 0 0" rpy="0 0 0"/>
         <mass value="0.001"/>
-        <inertia ixx="0.00001" ixy="0" ixz="0"
-                 iyy="0.00001" iyz="0"
-                 izz="0.00001"/>
+        <inertia ixx="0.00001" ixy="0" ixz="0" iyy="0.00001" iyz="0" izz="0.00001"/>
       </inertial>
     </link>
@@ -79,7 +76,5 @@
         <origin xyz="0 0 0" rpy="0 0 0"/>
         <mass value="0.001"/>
-        <inertia ixx="0.00001" ixy="0" ixz="0"
-                 iyy="0.00001" iyz="0"
-                 izz="0.00001"/>
+        <inertia ixx="0.00001" ixy="0" ixz="0" iyy="0.00001" iyz="0" izz="0.00001"/>
       </inertial>
     </link>
@@ -94,7 +89,5 @@
         <origin xyz="0 0 0" rpy="0 0 0"/>
         <mass value="0.001"/>
-        <inertia ixx="0.00001" ixy="0" ixz="0"
-                 iyy="0.00001" iyz="0"
-                 izz="0.00001"/>
+        <inertia ixx="0.00001" ixy="0" ixz="0" iyy="0.00001" iyz="0" izz="0.00001"/>
       </inertial>
     </link>
@@ -108,7 +101,5 @@
         <origin xyz="0 0 0" rpy="0 0 0"/>
         <mass value="0.001"/>
-        <inertia ixx="0.00001" ixy="0" ixz="0"
-                 iyy="0.00001" iyz="0"
-                 izz="0.00001"/>
+        <inertia ixx="0.00001" ixy="0" ixz="0" iyy="0.00001" iyz="0" izz="0.00001"/>
       </inertial>
     </link>
@@ -123,7 +114,5 @@
         <origin xyz="0 0 0" rpy="0 0 0"/>
         <mass value="0.001"/>
-        <inertia ixx="0.00001" ixy="0" ixz="0"
-                 iyy="0.00001" iyz="0"
-                 izz="0.00001"/>
+        <inertia ixx="0.00001" ixy="0" ixz="0" iyy="0.00001" iyz="0" izz="0.00001"/>
       </inertial>
     </link>
@@ -137,10 +126,8 @@
         <origin xyz="0 0 0" rpy="0 0 0"/>
         <mass value="0.001"/>
-        <inertia ixx="0.00001" ixy="0" ixz="0"
-                 iyy="0.00001" iyz="0"
-                 izz="0.00001"/>
+        <inertia ixx="0.00001" ixy="0" ixz="0" iyy="0.00001" iyz="0" izz="0.00001"/>
       </inertial>
     </link>
-    <!-- extensions -->
+    <!-- Gazebo config -->
     <xacro:openni_camera_gazebo_v0 name="${name}" />
   </xacro:macro>

File: tiago_description/urdf/sensors/xtion_pro_live.urdf.xacro (robot description, xacro)
@@ -1,5 +1,5 @@
 <?xml version="1.0"?>
 <!--
-  Copyright (c) 2022 PAL Robotics S.L. All rights reserved.
+  Copyright (c) 2024 PAL Robotics S.L. All rights reserved.
   Licensed under the Apache License, Version 2.0 (the "License");
   you may not use this file except in compliance with the License.
@@ -13,8 +13,9 @@
  -->
 <robot xmlns:xacro="http://ros.org/wiki/xacro">
+  <!-- INCLUDES -->
   <xacro:include filename="$(find tiago_description)/urdf/sensors/openni.gazebo.xacro" />
-  <!-- Macro -->
+  <!-- MACRO DEFINITION-->
   <xacro:macro name="xtion_pro_live" params="name parent camera_model *origin *optical_origin extrinsic_calibration_dir">
-    <!-- includes -->
+    <!-- INCLUDES -->
     <xacro:include filename="${extrinsic_calibration_dir}/extrinsic_camera_calibration_constants.urdf.xacro" />
     <!-- frames in the center of the camera -->
@@ -28,7 +29,5 @@
         <origin xyz="-0.00936000000 -0.00003000000 -0.00273000000" rpy="0 0 0"/>
         <mass value="0.21970000000"/>
-        <inertia ixx="0.00000429247" ixy="0.00000000000" ixz="0.00000002565"
-                 iyy="0.00000008027" iyz="0.00000000000"
-                 izz="0.00000427339"/>
+        <inertia ixx="0.00000429247" ixy="0.00000000000" ixz="0.00000002565" iyy="0.00000008027" iyz="0.00000000000" izz="0.00000427339"/>
       </inertial>
       <!--
@@ -59,7 +58,5 @@
         <origin xyz="0 0 0" rpy="0 0 0"/>
         <mass value="0.001"/>
-        <inertia ixx="0.00001" ixy="0" ixz="0"
-                 iyy="0.00001" iyz="0"
-                 izz="0.00001"/>
+        <inertia ixx="0.00001" ixy="0" ixz="0" iyy="0.00001" iyz="0" izz="0.00001"/>
       </inertial>
     </link>
@@ -74,7 +71,5 @@
         <origin xyz="0 0 0" rpy="0 0 0"/>
         <mass value="0.001"/>
-        <inertia ixx="0.00001" ixy="0" ixz="0"
-                 iyy="0.00001" iyz="0"
-                 izz="0.00001"/>
+        <inertia ixx="0.00001" ixy="0" ixz="0" iyy="0.00001" iyz="0" izz="0.00001"/>
       </inertial>
     </link>
@@ -88,7 +83,5 @@
         <origin xyz="0 0 0" rpy="0 0 0"/>
         <mass value="0.001"/>
-        <inertia ixx="0.00001" ixy="0" ixz="0"
-                 iyy="0.00001" iyz="0"
-                 izz="0.00001"/>
+        <inertia ixx="0.00001" ixy="0" ixz="0" iyy="0.00001" iyz="0" izz="0.00001"/>
       </inertial>
     </link>
@@ -103,7 +96,5 @@
         <origin xyz="0 0 0" rpy="0 0 0"/>
         <mass value="0.001"/>
-        <inertia ixx="0.00001" ixy="0" ixz="0"
-                 iyy="0.00001" iyz="0"
-                 izz="0.00001"/>
+        <inertia ixx="0.00001" ixy="0" ixz="0" iyy="0.00001" iyz="0" izz="0.00001"/>
       </inertial>
     </link>
@@ -117,10 +108,8 @@
         <origin xyz="0 0 0" rpy="0 0 0"/>
         <mass value="0.001"/>
-        <inertia ixx="0.00001" ixy="0" ixz="0"
-                 iyy="0.00001" iyz="0"
-                 izz="0.00001"/>
+        <inertia ixx="0.00001" ixy="0" ixz="0" iyy="0.00001" iyz="0" izz="0.00001"/>
       </inertial>
     </link>
-    <!-- extensions -->
+    <!-- Gazebo -->
     <xacro:openni_camera_gazebo_v0 name="${name}" />
   </xacro:macro>
