Commit message: ROS2 control and include std

File: tiago_description/robots/tiago.urdf.xacro (robot description, xacro)
@@ -123,6 +123,4 @@
   <!-- Tools -->
   <xacro:include filename="$(find pal_urdf_utils)/urdf/deg_to_rad.urdf.xacro" />
-  <!-- Calibration constants -->
-  <xacro:include filename="${description_calibration_dir}/calibration_constants.urdf.xacro" />
   <!-- Materials for visualization -->
   <xacro:include filename="$(find pal_urdf_utils)/urdf/materials.urdf.xacro" />
@@ -188,4 +186,4 @@
   </link>
   <!-- ROS 2 Control -->
-  <xacro:tiago_ros2_control use_sim="$(arg use_sim)" />
+  <xacro:tiago_ros2_control />
 </robot>

File: tiago_description/ros2_control/ros2_control.urdf.xacro (robot description, xacro)
@@ -13,17 +13,13 @@
  -->
 <robot xmlns:xacro="http://ros.org/wiki/xacro" name="tiago">
-  <xacro:macro name="tiago_ros2_control" params="use_sim:=^|false">
-    <xacro:arg name="arm_model" default="tiago-arm" />
-    <xacro:arg name="end_effector" default="pal-hey5"/>
-    <xacro:arg name="description_calibration_dir" default="$(find tiago_description)/urdf/calibration" />
-    <xacro:property name="has_arm" value="${arm_model not in ['no-arm']}"/>
-    <xacro:property name="has_ft_sensor" value="${ft_sensor not in ['no-ft-sensor'] and has_arm}"/>
-    <xacro:property name="has_end_effector" value="${end_effector not in ['no-end-effector'] and has_arm}"/>
-    <xacro:property name="has_ft_sensor" value="${ft_sensor not in ['no-ft-sensor'] and has_arm}"/>
-    <xacro:include filename="$(find ${base_type}_description)/urdf/wheels/wheel.ros2_control.xacro" />
-    <xacro:include filename="$(find tiago_description)/urdf/torso/torso.ros2_control.xacro" />
-    <xacro:include filename="$(find tiago_description)/urdf/head/head.ros2_control.xacro" />
-    <xacro:include filename="$(find ${base_type}_description)/urdf/sensors/sensors.ros2_control.xacro"/>
-    <xacro:include filename="$(arg description_calibration_dir)/calibration_constants.urdf.xacro" />
+  <!-- INCLUDES -->
+  <xacro:include filename="$(find tiago_description)/urdf/torso/torso.ros2_control.xacro" />
+  <xacro:include filename="$(find tiago_description)/urdf/head/head.ros2_control.xacro" />
+  <xacro:include filename="$(find ${base_type}_description)/urdf/wheels/wheel.ros2_control.xacro" />
+  <!-- sensors.ros2_control.xacro should be separated into specific files-->
+  <xacro:include filename="$(find ${base_type}_description)/urdf/sensors/sensors.ros2_control.xacro"/>
+  <xacro:include filename="$(arg description_calibration_dir)/calibration_constants.urdf.xacro" />
+  <!-- MACRO DEFINITION-->
+  <xacro:macro name="tiago_ros2_control">
     <xacro:if value="${has_arm}">
       <xacro:include filename="$(find tiago_description)/urdf/arm/arm.ros2_control.xacro" />
@@ -39,14 +35,16 @@
       </xacro:if>
     </xacro:if>
+    <!-- ROS 2 config-->
     <ros2_control name="ros2_control_tiago_system" type="system">
+      <!-- Execution env config -->
       <hardware>
-        <xacro:if value="$(arg use_sim)">
+        <xacro:if value="${use_sim_time}">
           <plugin>gazebo_ros2_control/GazeboSystem</plugin>
         </xacro:if>
-        <xacro:unless value="$(arg use_sim)">
+        <xacro:unless value="${use_sim_time}">
           <plugin>robot_control/RobotControl</plugin>
         </xacro:unless>
       </hardware>
-      <!-- wheels -->
+      <!-- Wheels -->
       <xacro:if value="${base_type == 'pmb2'}">
         <xacro:ros2_control_wheel side="right" />
@@ -60,12 +58,10 @@
       </xacro:if>
       <!-- IMU -->
-      <xacro:if value="$(arg use_sim)">
+      <xacro:if value="${use_sim_time}">
         <xacro:ros2_control_imu name="base_imu_sensor"/>
       </xacro:if>
-      <!-- torso -->
+      <!-- Torso -->
       <xacro:ros2_control_torso name="torso_lift" reduction="1.0" />
-      <!-- head -->
-      <xacro:ros2_control_head name="head_1" reduction="1.0" offset="${head_1_joint_offset}" />
-      <xacro:ros2_control_head name="head_2" reduction="1.0" offset="${head_2_joint_offset}" />
+      <!-- arm -->
       <xacro:if value="${has_arm}">
         <!-- arm -->
@@ -79,18 +75,14 @@
         <!-- End effector -->
         <xacro:if value="${end_effector == 'pal-gripper'}">
-          <!-- pal-gripper -->
           <xacro:ros2_control_gripper name="gripper_left_finger" reduction="1.0" />
           <xacro:ros2_control_gripper name="gripper_right_finger" reduction="1.0" />
         </xacro:if>
         <xacro:if value="${end_effector == 'pal-hey5'}">
-          <!-- pal-hey5 -->
           <xacro:ros2_control_hey5 name="hand"/>
         </xacro:if>
         <xacro:if value="${end_effector == 'robotiq-2f-85'}">
-          <!-- robotiq-2f-85 -->
           <xacro:ros2_control_robotiq_85_gripper name="gripper" reduction="1.0" />
         </xacro:if>
         <xacro:if value="${end_effector == 'robotiq-2f-140'}">
-          <!-- robotiq-2f-140 -->
           <xacro:ros2_control_robotiq_140_gripper name="gripper" reduction="1.0" />
         </xacro:if>
@@ -101,4 +93,7 @@
         <xacro:ros2_control_force_torque_sensor name="wrist_ft_sensor"/>
       </xacro:if>
+      <!-- Head -->
+      <xacro:ros2_control_head name="head_1" reduction="1.0" offset="${head_1_joint_offset}" />
+      <xacro:ros2_control_head name="head_2" reduction="1.0" offset="${head_2_joint_offset}" />
     </ros2_control>
   </xacro:macro>

File: tiago_description/urdf/head/head.urdf.xacro (robot description, xacro)
@@ -25,4 +25,5 @@
   <xacro:include filename="$(find tiago_description)/urdf/sensors/xtion_pro_live.urdf.xacro" />
   <xacro:include filename="$(find tiago_description)/urdf/sensors/orbbec_astra.urdf.xacro" />
+  <xacro:include filename="$(arg description_calibration_dir)/calibration_constants.urdf.xacro" />
   <!-- MACRO DEFINITION-->
   <!-- head_1 (pan) -->
@@ -102,6 +103,4 @@
     <!-- PROPERTIES -->
     <xacro:property name="head_eps" value="${0.00 if no_safety_eps else 0.07}" />
-    <!-- INCLUDES -->
-    <xacro:include filename="$(arg description_calibration_dir)/calibration_constants.urdf.xacro" />
     <!-- HEAD DEFINITION -->
     <!-- Head links -->

File: tiago_description/urdf/sensors/openni.gazebo.xacro (robot description, xacro)
@@ -1,5 +1,5 @@
 <?xml version="1.0"?>
 <!--
-  Copyright (c) 2022 PAL Robotics S.L. All rights reserved.
+  Copyright (c) 2024 PAL Robotics S.L. All rights reserved.
   Licensed under the Apache License, Version 2.0 (the "License");
   you may not use this file except in compliance with the License.

File: tiago_description/urdf/sensors/orbbec_astra.urdf.xacro (robot description, xacro)
@@ -16,8 +16,7 @@
   <!-- INCLUDES -->
   <xacro:include filename="$(find tiago_description)/urdf/sensors/openni.gazebo.xacro" />
+  <xacro:include filename="${extrinsic_calibration_dir}/extrinsic_camera_calibration_constants.urdf.xacro" />
   <!-- MACRO DEFINITION-->
   <xacro:macro name="orbbec_astra" params="name parent camera_model *origin *optical_origin extrinsic_calibration_dir">
-    <!-- INCLUDES -->
-    <xacro:include filename="${extrinsic_calibration_dir}/extrinsic_camera_calibration_constants.urdf.xacro" />
     <!-- frames in the center of the camera -->
     <joint name="${name}_joint" type="fixed">

File: tiago_description/urdf/sensors/xtion_pro_live.urdf.xacro (robot description, xacro)
@@ -15,8 +15,7 @@
   <!-- INCLUDES -->
   <xacro:include filename="$(find tiago_description)/urdf/sensors/openni.gazebo.xacro" />
+  <xacro:include filename="${extrinsic_calibration_dir}/extrinsic_camera_calibration_constants.urdf.xacro" />
   <!-- MACRO DEFINITION-->
   <xacro:macro name="xtion_pro_live" params="name parent camera_model *origin *optical_origin extrinsic_calibration_dir">
-    <!-- INCLUDES -->
-    <xacro:include filename="${extrinsic_calibration_dir}/extrinsic_camera_calibration_constants.urdf.xacro" />
     <!-- frames in the center of the camera -->
     <joint name="${name}_joint" type="fixed">

File: tiago_description/urdf/torso/torso.ros2_control.xacro (robot description, xacro)
@@ -13,5 +13,5 @@
  -->
 <robot xmlns:xacro="http://ros.org/wiki/xacro">
-  <xacro:macro name="ros2_control_torso" params="name reduction" >
+  <xacro:macro name="ros2_control_torso" params="name reduction">
     <joint name="${name}_joint">
       <command_interface name="position" />
