Commit message: Arm std

File: tiago_description/urdf/arm/wrist.urdf.xacro (robot description, xacro)
@@ -1,5 +1,5 @@
 <?xml version="1.0"?>
 <!--
-  Copyright (c) 2022 PAL Robotics S.L. All rights reserved.
+  Copyright (c) 2024 PAL Robotics S.L. All rights reserved.
   Licensed under the Apache License, Version 2.0 (the "License");
   you may not use this file except in compliance with the License.
@@ -13,20 +13,25 @@
  -->
 <robot xmlns:xacro="http://ros.org/wiki/xacro">
-  <!--File includes-->
+  <!-- INCLUDES -->
   <xacro:include filename="$(find pal_urdf_utils)/urdf/deg_to_rad.urdf.xacro" />
-  <!--Constant parameters-->
-  <xacro:property name="wrist_friction"       value="1.0" />
-  <xacro:property name="wrist_damping"        value="1.0" />
-  <xacro:property name="wrist_1_max_vel"      value="1.95" />
-  <xacro:property name="wrist_2_max_vel"      value="1.76" />
-  <xacro:property name="wrist_3_max_vel"      value="1.76" />
-  <xacro:property name="wrist_1_max_effort"   value="3" />
-  <xacro:property name="wrist_2_max_effort"   value="6.6" />
-  <xacro:property name="wrist_3_max_effort"   value="6.6" />
-  <xacro:macro name="wrist" params="name parent reflect wrist_model has_ft_sensor arm_5_offset arm_6_offset arm_7_offset no_safety_eps:=False">
-   <xacro:property name="wrist_eps"       value="${0.00 if no_safety_eps else 0.02}"/>
-    <!--************************-->
-    <!--        WRIST           -->
-    <!--************************-->
+  <!-- PROPERTIES -->
+  <xacro:property name="wrist_friction" value="1.0" />
+  <xacro:property name="wrist_damping" value="1.0" />
+  <xacro:property name="wrist_1_max_vel" value="1.95" />
+  <xacro:property name="wrist_2_max_vel" value="1.76" />
+  <xacro:property name="wrist_3_max_vel" value="1.76" />
+  <xacro:property name="wrist_1_max_effort" value="3" />
+  <xacro:property name="wrist_2_max_effort" value="6.6" />
+  <xacro:property name="wrist_3_max_effort" value="6.6" />
+  <xacro:property name="wrist_eps" value="${0.00 if no_safety_eps else 0.02}"/>
+  <xacro:if value="${wrist_model == 'wrist-2010'}">
+    <xacro:property name="wrist_6_range" value="${ 81 if has_ft_sensor else 90 }"/>
+  </xacro:if>
+  <xacro:if value="${wrist_model == 'wrist-2017'}">
+    <xacro:property name="wrist_6_range" value="81"/>
+  </xacro:if>
+  <!-- MACRO DEFINITION -->
+  <xacro:macro name="wrist" params="name parent reflect">
+    <!-- Wrist-->
     <link name="${name}_5_link">
       <inertial>
@@ -34,13 +39,9 @@
         <xacro:if value="${wrist_model == 'wrist-2010'}">
           <mass value="1.655819"/>
-          <inertia ixx="0.00613800000" ixy="-0.00000400000" ixz="0.00015600000"
-                   iyy="0.00564000000" iyz="0.00002200000"
-                   izz="0.00179700000"/>
+          <inertia ixx="0.00613800000" ixy="-0.00000400000" ixz="0.00015600000" iyy="0.00564000000" iyz="0.00002200000" izz="0.00179700000"/>
         </xacro:if>
         <xacro:if value="${wrist_model == 'wrist-2017'}">
           <mass value="0.9359143689" />
-          <inertia ixx="0.001036187977" ixy="1.0622321E-07" ixz="1.9920336E-06"
-                   iyy="0.000794527176366096" iyz="-2.56396106998404E-07"
-                   izz="0.000439831229979178" />
+          <inertia ixx="0.001036187977" ixy="1.0622321E-07" ixz="1.9920336E-06" iyy="0.000794527176366096" iyz="-2.56396106998404E-07" izz="0.000439831229979178" />
         </xacro:if>
       </inertial>
@@ -66,8 +67,5 @@
       <limit lower="${-120.0 * deg_to_rad}" upper="${120.0 * deg_to_rad}" effort="${wrist_1_max_effort}" velocity="${wrist_1_max_vel}" />
       <dynamics friction="${wrist_friction}" damping="${wrist_damping}"/>
-      <safety_controller k_position="20"
-                         k_velocity="20"
-                         soft_lower_limit="${-120.0 * deg_to_rad + wrist_eps}"
-                         soft_upper_limit="${ 120.0 * deg_to_rad - wrist_eps}" />
+      <safety_controller k_position="20" k_velocity="20" soft_lower_limit="${-120.0 * deg_to_rad + wrist_eps}" soft_upper_limit="${ 120.0 * deg_to_rad - wrist_eps}" />
     </joint>
     <link name="${name}_6_link">
@@ -76,13 +74,9 @@
         <xacro:if value="${wrist_model == 'wrist-2010'}">
           <mass value="0.370063"/>
-          <inertia ixx="0.00021500000" ixy="0.00000000000" ixz="0.00000000000"
-                   iyy="0.00017000000" iyz="0.00000200000"
-                   izz="0.00017400000"/>
+          <inertia ixx="0.00021500000" ixy="0.00000000000" ixz="0.00000000000" iyy="0.00017000000" iyz="0.00000200000" izz="0.00017400000"/>
         </xacro:if>
         <xacro:if value="${wrist_model == 'wrist-2017'}">
           <mass value="0.30275767222" />
-          <inertia ixx="3.29233557E-05" ixy="6.31537395E-08" ixz="-4.567124912E-11"
-                   iyy="3.85334410118923E-05" iyz="-2.01613082836742E-07"
-                   izz="3.33282849168039E-05" />
+          <inertia ixx="3.29233557E-05" ixy="6.31537395E-08" ixz="-4.567124912E-11" iyy="3.85334410118923E-05" iyz="-2.01613082836742E-07" izz="3.33282849168039E-05" />
         </xacro:if>
       </inertial>
@@ -101,10 +95,4 @@
       </collision>
     </link>
-    <xacro:if value="${wrist_model == 'wrist-2010'}">
-      <xacro:property name="wrist_6_range"           value="${ 81 if has_ft_sensor else 90 }"/>
-    </xacro:if>
-    <xacro:if value="${wrist_model == 'wrist-2017'}">
-      <xacro:property name="wrist_6_range"           value="81"/>
-    </xacro:if>
     <joint name="${name}_6_joint" type="revolute">
       <parent link="${name}_5_link" />
@@ -114,8 +102,5 @@
       <limit lower="${-wrist_6_range * deg_to_rad}" upper="${wrist_6_range * deg_to_rad}" effort="${wrist_2_max_effort}" velocity="${wrist_2_max_vel}" />
       <dynamics friction="${wrist_friction}" damping="${wrist_damping}"/>
-      <safety_controller k_position="20"
-                         k_velocity="20"
-                         soft_lower_limit="${-wrist_6_range * deg_to_rad + wrist_eps}"
-                         soft_upper_limit="${ wrist_6_range * deg_to_rad - wrist_eps}" />
+      <safety_controller k_position="20" k_velocity="20" soft_lower_limit="${-wrist_6_range * deg_to_rad + wrist_eps}" soft_upper_limit="${ wrist_6_range * deg_to_rad - wrist_eps}" />
     </joint>
     <link name="${name}_7_link">
@@ -124,13 +109,9 @@
         <xacro:if value="${wrist_model == 'wrist-2010'}">
           <mass value="0.234252"/>
-          <inertia ixx="0.00014200000" ixy="0.00000000000" ixz="0.00000000000"
-                   iyy="0.00011300000" iyz="0.00000000000"
-                   izz="0.00005200000"/>
+          <inertia ixx="0.00014200000" ixy="0.00000000000" ixz="0.00000000000" iyy="0.00011300000" iyz="0.00000000000" izz="0.00005200000"/>
         </xacro:if>
         <xacro:if value="${wrist_model == 'wrist-2017'}">
           <mass value="0.100" />
-          <inertia ixx="1.14959795E-05" ixy="-1.390727219E-07" ixz="5.930207406E-09"
-                   iyy="1.13594084240734E-05" iyz="-1.78396260812528E-08"
-                   izz="2.01898984804048E-05" />
+          <inertia ixx="1.14959795E-05" ixy="-1.390727219E-07" ixz="5.930207406E-09" iyy="1.13594084240734E-05" iyz="-1.78396260812528E-08" izz="2.01898984804048E-05" />
         </xacro:if>
       </inertial>
@@ -143,8 +124,5 @@
       <limit lower="${-120.0 * deg_to_rad}" upper="${120.0 * deg_to_rad}" effort="${wrist_3_max_effort}" velocity="${wrist_3_max_vel}" />
       <dynamics friction="${wrist_friction}" damping="${wrist_damping}"/>
-      <safety_controller k_position="20"
-                         k_velocity="20"
-                         soft_lower_limit="${-120.0 * deg_to_rad + wrist_eps}"
-                         soft_upper_limit="${ 120.0 * deg_to_rad - wrist_eps}" />
+      <safety_controller k_position="20" k_velocity="20" soft_lower_limit="${-120.0 * deg_to_rad + wrist_eps}" soft_upper_limit="${ 120.0 * deg_to_rad - wrist_eps}" />
     </joint>
     <gazebo reference="${name}_5_link">
@@ -161,12 +139,12 @@
     </gazebo>
     <gazebo reference="${name}_5_joint">
-        <implicitSpringDamper>1</implicitSpringDamper>
+      <implicitSpringDamper>1</implicitSpringDamper>
     </gazebo>
     <gazebo reference="${name}_6_joint">
-        <implicitSpringDamper>1</implicitSpringDamper>
+      <implicitSpringDamper>1</implicitSpringDamper>
     </gazebo>
     <gazebo reference="${name}_7_joint">
-        <implicitSpringDamper>1</implicitSpringDamper>
-        <provideFeedback>1</provideFeedback>
+      <implicitSpringDamper>1</implicitSpringDamper>
+      <provideFeedback>1</provideFeedback>
     </gazebo>
   </xacro:macro>

Commit message: ee std

File: tiago_description/robots/tiago.urdf.xacro (robot description, xacro)
@@ -149,5 +149,5 @@
     <!-- End effector -->
     <xacro:if value="${has_end_effector}">
-      <xacro:tiago_end_effector name="${end_effector_name}" parent="${end_effector_link}" type="${end_effector}" reflect="1"/>
+      <xacro:tiago_end_effector name="${end_effector_name}" parent="${end_effector_link}" reflect="1"/>
     </xacro:if>
     <!-- FT sensor -->

File: tiago_description/urdf/end_effector/end_effector.urdf.xacro (robot description, xacro)
@@ -1,5 +1,5 @@
 <?xml version="1.0"?>
 <!--
-  Copyright (c) 2022 PAL Robotics S.L. All rights reserved.
+  Copyright (c) 2024 PAL Robotics S.L. All rights reserved.
   Licensed under the Apache License, Version 2.0 (the "License");
   you may not use this file except in compliance with the License.
@@ -13,60 +13,53 @@
  -->
 <robot xmlns:xacro="http://ros.org/wiki/xacro">
-  <!--File includes-->
+  <!-- INCLUDES -->
   <xacro:include filename="$(find pal_urdf_utils)/urdf/deg_to_rad.urdf.xacro" />
   <xacro:include filename="$(find pal_hey5_description)/urdf/pal_hey5_hand.urdf.xacro" />
-  <!--
-    Utiliy to create a tiago end effector (right or left).
-    Parameters:
-    - name: End effector name. The created links and joints are prepended with 'name_'
-    - parent: Parent link
-    - reflect: Set to 1 for a right end effector, or to -1 for a left end effector
-  -->
-  <xacro:macro name="tiago_end_effector" params="name parent type reflect tiago_dual:=false">
-  <!-- PAL Gripper -->
-  <xacro:if value="${type == 'pal-gripper'}">
-    <xacro:include filename="$(find pal_gripper_description)/urdf/gripper.urdf.xacro" />
-    <xacro:pal_gripper parent="${parent}" name="${name}">
-      <origin xyz="0.01 0 0" rpy="${90*deg_to_rad} ${90*deg_to_rad} ${-90*deg_to_rad}"/>
-    </xacro:pal_gripper>
+  <xacro:if value="${end_effector == 'pal-gripper'}">
+    <xacro:include filename="$(find pal_gripper_description)/urdf/gripper.ros2_control.xacro" />
   </xacro:if>
-  <!-- Robotiq 2F-85 Gripper -->
-  <xacro:if value="${type == 'robotiq-2f-85'}">
-    <xacro:include filename="$(find pal_robotiq_description)/urdf/robotiq_85_gripper.urdf.xacro" />
-    <xacro:robotiq_85_gripper prefix="${name}_" parent="${parent}" >
-      <origin xyz="0.01 0 0" rpy="${90*deg_to_rad} ${0*deg_to_rad} ${90*deg_to_rad}"/>
-    </xacro:robotiq_85_gripper>
+  <xacro:if value="${end_effector == 'pal-hey5'}">
+    <xacro:include filename="$(find pal_hey5_description)/urdf/pal_hey5.ros2_control.xacro" />
   </xacro:if>
-  <!-- Robotiq 2F-140 Gripper -->
-  <xacro:if value="${type == 'robotiq-2f-140'}">
-    <xacro:include filename="$(find pal_robotiq_description)/urdf/robotiq_140_gripper.urdf.xacro" />
-    <xacro:robotiq_140_gripper prefix="${name}_" parent="${parent}" >
-      <origin xyz="0.01 0 0" rpy="${90*deg_to_rad} ${0*deg_to_rad} ${90*deg_to_rad}"/>
-    </xacro:robotiq_140_gripper>
+  <xacro:if value="${end_effector in ['robotiq-2f-85', 'robotiq-2f-140']}">
+    <xacro:include filename="$(find pal_robotiq_description)/urdf/robotiq.ros2_control.xacro" />
   </xacro:if>
-  <!-- Robotiq Epick Gripper -->
-  <!-- <xacro:if value="${type == 'robotiq-epick'}">
-    <xacro:include filename="$(find pal_robotiq_epick_description)/urdf/robotiq_epick_model_macro.xacro" />
-    <xacro:epick_hand  prefix="${name}_" parent="${parent}">
-      <origin xyz="0.01 0 0" rpy="${90*deg_to_rad} ${0*deg_to_rad} ${90*deg_to_rad}"/>
-    </xacro:epick_hand>
-  </xacro:if> -->
-  <!-- Hand -->
-  <xacro:if value="${type == 'pal-hey5'}">
-    <xacro:pal_hey5_hand parent="${parent}" name="${name}" reflect="${reflect}">
-      <origin xyz="0 0 0" rpy="0 0 0"/>
-    </xacro:pal_hey5_hand>
-    <joint name="${name}_safety_box_joint" type="fixed">
-      <parent link="${parent}"/>
-      <child link="${name}_safety_box"/>
-      <origin xyz="0.1 0.02 ${reflect * 0.02}" rpy="0 0 0"/>
-    </joint>
-    <link name="${name}_safety_box">
-      <inertial>
+  <!-- MACRO DEFINITION -->
+  <xacro:macro name="tiago_end_effector" params="name parent reflect tiago_dual:=false">
+    <!-- PAL Gripper -->
+    <xacro:if value="${end_effector == 'pal-gripper'}">
+      <xacro:pal_gripper parent="${parent}" name="${name}">
+        <origin xyz="0.01 0 0" rpy="${90*deg_to_rad} ${90*deg_to_rad} ${-90*deg_to_rad}"/>
+      </xacro:pal_gripper>
+    </xacro:if>
+    <!-- Robotiq 2F-85 Gripper -->
+    <xacro:if value="${end_effector == 'robotiq-2f-85'}">
+      <xacro:robotiq_85_gripper prefix="${name}_" parent="${parent}">
+        <origin xyz="0.01 0 0" rpy="${90*deg_to_rad} ${0*deg_to_rad} ${90*deg_to_rad}"/>
+      </xacro:robotiq_85_gripper>
+    </xacro:if>
+    <!-- Robotiq 2F-140 Gripper -->
+    <xacro:if value="${end_effector == 'robotiq-2f-140'}">
+      <xacro:robotiq_140_gripper prefix="${name}_" parent="${parent}">
+        <origin xyz="0.01 0 0" rpy="${90*deg_to_rad} ${0*deg_to_rad} ${90*deg_to_rad}"/>
+      </xacro:robotiq_140_gripper>
+    </xacro:if>
+    <!-- Hand -->
+    <xacro:if value="${end_effector == 'pal-hey5'}">
+      <xacro:pal_hey5_hand parent="${parent}" name="${name}" reflect="${reflect}">
         <origin xyz="0 0 0" rpy="0 0 0"/>
-        <mass value="0.0001" />
-        <inertia ixx="0.0001"  ixy="0"  ixz="0" iyy="0.0001" iyz="0" izz="0.0001" />
-      </inertial>
-      <!--
+      </xacro:pal_hey5_hand>
+      <joint name="${name}_safety_box_joint" type="fixed">
+        <parent link="${parent}"/>
+        <child link="${name}_safety_box"/>
+        <origin xyz="0.1 0.02 ${reflect * 0.02}" rpy="0 0 0"/>
+      </joint>
+      <link name="${name}_safety_box">
+        <inertial>
+          <origin xyz="0 0 0" rpy="0 0 0"/>
+          <mass value="0.0001" />
+          <inertia ixx="0.0001" ixy="0" ixz="0" iyy="0.0001" iyz="0" izz="0.0001" />
+        </inertial>
+        <!--
       <visual>
         <origin xyz="0 0 0" rpy="0 0 0" />
@@ -76,22 +69,22 @@
       </visual>
       -->
-      <collision>
-        <origin xyz="0 0 0" rpy="0 0 0" />
-        <geometry>
-          <box size="0.2 0.115 0.18" />
-        </geometry>
-      </collision>
-    </link>
-  </xacro:if>
-  <!-- Custom -->
-  <!--xacro:if value="${type == 'custom' and not tiago_dual}">
+        <collision>
+          <origin xyz="0 0 0" rpy="0 0 0" />
+          <geometry>
+            <box size="0.2 0.115 0.18" />
+          </geometry>
+        </collision>
+      </link>
+    </xacro:if>
+    <!-- Custom -->
+    <!--xacro:if value="${end_effector == 'custom' and not tiago_dual}">
     <xacro:include filename="$(find custom_ee_description)/urdf/end-effector.urdf.xacro" />
-    <xacro:end_effector parent="${parent}">
-      <origin xyz="0.01 0 0" rpy="${90*deg_to_rad} ${90*deg_to_rad} ${-90*deg_to_rad}"/>
-    </xacro:end_effector>
-  </xacro:if-->
-  <!-- Custom dual-->
-  <!--xacro:if value="${type == 'custom' and tiago_dual}">
-    <xacro:if value="${reflect == 1}"--> <!-- If right -->
+      <xacro:end_effector parent="${parent}">
+        <origin xyz="0.01 0 0" rpy="${90*deg_to_rad} ${90*deg_to_rad} ${-90*deg_to_rad}"/>
+      </xacro:end_effector>
+    </xacro:if-->
+    <!-- Custom dual-->
+    <!--xacro:if value="${end_effector == 'custom' and tiago_dual}">
+      <xacro:if value="${reflect == 1}"-->    <!-- If right -->
     <!--xacro:include filename="$(find custom_dual_ee_description)/urdf/end-effector-right.urdf.xacro" />
     <xacro:end_effector_right parent="${parent}">
@@ -99,5 +92,5 @@
     </xacro:end_effector_right>
     </xacro:if>
-    <xacro:if value="${reflect == -1}"--> <!-- If left -->
+    <xacro:if value="${reflect == -1}"-->    <!-- If left -->
     <!--xacro:include filename="$(find custom_dual_ee_description)/urdf/end-effector-left.urdf.xacro" />
     <xacro:end_effector_left parent="${parent}">

Commit message: FT sensor std

File: tiago_description/robots/tiago.urdf.xacro (robot description, xacro)
@@ -57,5 +57,4 @@
   <xacro:property name="end_effector" value="$(arg end_effector)" />
   <xacro:property name="camera_model" value="$(arg camera_model)" />
-  <xacro:property name="head_link_name" value="head_2_link"/>
   <xacro:property name="no_safety_eps" value="$(arg no_safety_eps)" />
   <!-- HW configuration check -->
@@ -113,5 +112,4 @@
   <xacro:if value="${has_ft_sensor}">
     <xacro:include filename="$(find tiago_description)/urdf/sensors/ftsensor.urdf.xacro" />
-    <xacro:include filename="$(find tiago_description)/urdf/sensors/ftsensor.gazebo.xacro" />
   </xacro:if>
   <!-- End effector -->
@@ -154,21 +152,5 @@
     <xacro:if value="${has_ft_sensor}">
       <xacro:ft_sensor name="wrist" parent="arm_tool_link" />
-      <xacro:force_torque_sensor_gazebo name="wrist_ft" update_rate="100"/>
     </xacro:if>
-  </xacro:if>
-  <!-- Thermal camera -->
-  <xacro:if value="$(arg has_thermal_camera)">
-    <joint name="thermal_camera_joint" type="fixed">
-      <parent link="${head_link_name}"/>
-      <child link="thermal_camera"/>
-      <origin xyz="0.05 0.15 0" rpy="${0*deg_to_rad} ${-90*deg_to_rad} ${-180*deg_to_rad}" />
-    </joint>
-    <link name="thermal_camera">
-      <inertial>
-        <origin xyz="0 0 0" rpy="0 0 0"/>
-        <mass value="0.0001" />
-        <inertia ixx="0.0001" ixy="0" ixz="0" iyy="0.0001" iyz="0" izz="0.0001" />
-      </inertial>
-    </link>
   </xacro:if>
   <!-- RGBD Laser Link -->

File: tiago_description/ros2_control/ros2_control.urdf.xacro (robot description, xacro)
@@ -32,4 +32,7 @@
       <xacro:include filename="$(find pal_robotiq_description)/urdf/robotiq.ros2_control.xacro" />
     </xacro:if>
+  </xacro:if>
+  <xacro:if value="${has_ft_sensor}">
+    <xacro:include filename="$(find tiago_description)/urdf/sensors/ftsensor.ros2_control.xacro"/>
   </xacro:if>
   <!-- MACRO DEFINITION-->
@@ -75,5 +78,4 @@
         <!-- Force Torque sensor -->
         <xacro:if value="${has_ft_sensor}">
-          <xacro:include filename="$(find tiago_description)/urdf/sensors/sensors.ros2_control.xacro"/>
           <xacro:ros2_control_force_torque_sensor name="wrist_ft_sensor"/>
         </xacro:if>

File: tiago_description/urdf/sensors/ftsensor.gazebo.xacro (robot description, xacro)
@@ -1,5 +1,5 @@
 <?xml version="1.0"?>
 <!--
-  Copyright (c) 2022 PAL Robotics S.L. All rights reserved.
+  Copyright (c) 2024 PAL Robotics S.L. All rights reserved.
   Licensed under the Apache License, Version 2.0 (the "License");
   you may not use this file except in compliance with the License.
@@ -14,15 +14,15 @@
 <robot xmlns:xacro="http://ros.org/wiki/xacro">
   <xacro:macro name="force_torque_sensor_gazebo" params="name update_rate">
-  <gazebo reference="${name}_joint">
-    <preserveFixedJoint>true</preserveFixedJoint> <!-- in case this is in a fixed joint -->
-    <sensor name="${name}_sensor" type="force_torque">
-      <update_rate>${update_rate}</update_rate>
-      <visualize>true</visualize>
-      <force_torque>
-        <frame>child</frame>
-        <measure_direction>child_to_parent</measure_direction>
-      </force_torque>
-    </sensor>
-</gazebo>
-</xacro:macro>
+    <gazebo reference="${name}_joint">
+      <preserveFixedJoint>true</preserveFixedJoint>      <!-- in case this is in a fixed joint -->
+      <sensor name="${name}_sensor" type="force_torque">
+        <update_rate>${update_rate}</update_rate>
+        <visualize>true</visualize>
+        <force_torque>
+          <frame>child</frame>
+          <measure_direction>child_to_parent</measure_direction>
+        </force_torque>
+      </sensor>
+    </gazebo>
+  </xacro:macro>
 </robot>

Commit message: Thermal camera std

File: tiago_description/robots/tiago.urdf.xacro (robot description, xacro)
@@ -137,6 +137,4 @@
   <!-- Torso -->
   <xacro:tiago_torso name="torso" parent="base_link"/>
-  <!-- Head -->
-  <xacro:head name="head" parent="torso_lift_link" camera_model="${camera_model}" description_calibration_dir="${description_calibration_dir}" extrinsic_calibration_dir="${extrinsic_calibration_dir}" no_safety_eps="${no_safety_eps}"/>
   <!-- Arm -->
   <xacro:if value="${has_arm}">
@@ -145,13 +143,15 @@
       <origin xyz="0.15505 0.014 -0.151" rpy="0 0 ${-90 * deg_to_rad}" />
     </xacro:tiago_arm>
+    <!-- FT sensor -->
+    <xacro:if value="${has_ft_sensor}">
+      <xacro:ft_sensor name="wrist" parent="arm_tool_link" />
+    </xacro:if>
     <!-- End effector -->
     <xacro:if value="${has_end_effector}">
       <xacro:tiago_end_effector name="${end_effector_name}" parent="${end_effector_link}" reflect="1"/>
     </xacro:if>
-    <!-- FT sensor -->
-    <xacro:if value="${has_ft_sensor}">
-      <xacro:ft_sensor name="wrist" parent="arm_tool_link" />
-    </xacro:if>
   </xacro:if>
+  <!-- Head -->
+  <xacro:head name="head" parent="torso_lift_link"/>
   <!-- RGBD Laser Link -->
   <joint name="rgbd_laser_joint" type="fixed">

File: tiago_description/urdf/head/head.urdf.xacro (robot description, xacro)
@@ -14,4 +14,5 @@
 <robot xmlns:xacro="http://ros.org/wiki/xacro">
   <!-- PROPERTIES -->
+  <xacro:property name="head_link_name" value="head_2_link"/>
   <xacro:property name="head_friction" value="1.0" />
   <xacro:property name="head_damping" value="0.5" />
@@ -101,5 +102,5 @@
   </xacro:macro>
   <!-- Complete head -->
-  <xacro:macro name="head" params="name parent camera_model description_calibration_dir extrinsic_calibration_dir no_safety_eps:=False">
+  <xacro:macro name="head" params="name parent">
     <!-- Head links -->
     <xacro:head_1 name="${name}_1" parent="${parent}" />
@@ -122,4 +123,19 @@
       </xacro:orbbec_astra>
     </xacro:if>
+    <!-- Thermal camera -->
+    <xacro:if value="${has_thermal_camera}">
+      <joint name="thermal_camera_joint" type="fixed">
+        <parent link="${head_link_name}"/>
+        <child link="thermal_camera"/>
+        <origin xyz="0.05 0.15 0" rpy="${0*deg_to_rad} ${-90*deg_to_rad} ${-180*deg_to_rad}" />
+      </joint>
+      <link name="thermal_camera">
+        <inertial>
+          <origin xyz="0 0 0" rpy="0 0 0"/>
+          <mass value="0.0001" />
+          <inertia ixx="0.0001" ixy="0" ixz="0" iyy="0.0001" iyz="0" izz="0.0001" />
+        </inertial>
+      </link>
+    </xacro:if>
   </xacro:macro>
 </robot>
