Commit message: Final mods

File: tiago_description/robots/tiago.urdf.xacro (robot description, xacro)
@@ -16,6 +16,6 @@
   - Laser
   - Arm
+  - Wrist
   - FT Sensor
-  - Wrist
   - End effector
   - Camera
@@ -57,4 +57,5 @@
   <xacro:property name="end_effector" value="$(arg end_effector)" />
   <xacro:property name="camera_model" value="$(arg camera_model)" />
+  <xacro:property name="has_thermal_camera" default="$(arg has_thermal_camera)"/>
   <xacro:property name="no_safety_eps" value="$(arg no_safety_eps)" />
   <!-- HW configuration check -->
@@ -65,5 +66,5 @@
     <xacro:wrong_laser_model/>
   </xacro:if>
-  <xacro:if value="${arm_model not in ['tiago-arm', 'no-arm']}">
+  <xacro:if value="${arm_model not in ['no-arm', 'tiago-arm']}">
     <xacro:wrong_arm/>
   </xacro:if>
@@ -82,43 +83,43 @@
   <!-- HW configuration helpers-->
   <xacro:property name="has_arm" value="${arm_model != 'no-arm'}"/>
-  <xacro:property name="has_ft_sensor" value="${ft_sensor != 'no-ft-sensor' and has_arm}"/>
+  <xacro:property name="has_ft_sensor" value="${ft_sensor != 'no-ft-sensor'}"/>
   <xacro:property name="has_end_effector" value="${end_effector != 'no-end-effector'}"/>
   <xacro:property name="end_effector_link" value="${'wrist_ft_tool_link' if has_ft_sensor else 'arm_tool_link'}"/>
   <xacro:property name="end_effector_name" value="${'hand' if end_effector == 'pal-hey5' else 'gripper'}"/>
-  <xacro:property name="has_thermal_camera" default="$(arg has_thermal_camera)"/>
-  <xacro:property name="arm_x" default="0.08976" />
-  <xacro:property name="arm_y" default="0.15918" />
-  <xacro:property name="arm_z" default="-0.092008" />
-  <xacro:property name="arm_roll" default="-2.0679" />
-  <xacro:property name="arm_pitch" default="0.0" />
-  <xacro:property name="arm_yaw" default="-1.2217" />
+  <xacro:property name="arm_x" default="0.15505" />
+  <xacro:property name="arm_y" default="0.014" />
+  <xacro:property name="arm_z" default="-0.151" />
+  <xacro:property name="arm_roll" default="0" />
+  <xacro:property name="arm_pitch" default="0" />
+  <xacro:property name="arm_yaw" default="-90" />
   <!-- Calibration -->
   <xacro:property name="description_calibration_dir" value="$(arg description_calibration_dir)"/>
   <xacro:property name="extrinsic_calibration_dir" value="$(arg extrinsic_calibration_dir)"/>
   <!-- Execution env configuration -->
-  <xacro:property name="use_sim_time" default="$(arg is_multiple)"/>
+  <xacro:property name="use_sim_time" default="$(arg use_sim_time)"/>
   <xacro:property name="is_multiple" value="$(arg is_multiple)" />
   <xacro:property name="namespace" value="$(arg namespace)" />
   <!-- INCLUDES -->
+  <!-- Tools -->
+  <xacro:include filename="$(find pal_urdf_utils)/urdf/deg_to_rad.urdf.xacro" />
   <!-- Base -->
   <xacro:include filename="$(find ${base_type}_description)/urdf/base/base_sensors.urdf.xacro" />
   <!-- Torso -->
   <xacro:include filename="$(find tiago_description)/urdf/torso/torso.urdf.xacro" />
-  <!-- Arm -->
+  <!-- Arm, FT, EE -->
   <xacro:if value="${has_arm}">
+    <!-- Arm -->
     <xacro:include filename="$(find tiago_description)/urdf/arm/arm.urdf.xacro" />
-  </xacro:if>
-  <!-- Force Torque sensor -->
-  <xacro:if value="${has_ft_sensor}">
-    <xacro:include filename="$(find tiago_description)/urdf/sensors/ftsensor.urdf.xacro" />
-  </xacro:if>
-  <!-- End effector -->
-  <xacro:if value="${has_arm and has_end_effector}">
-    <xacro:include filename="$(find tiago_description)/urdf/end_effector/end_effector.urdf.xacro" />
+    <!-- FT sensor -->
+    <xacro:if value="${has_ft_sensor}">
+      <xacro:include filename="$(find tiago_description)/urdf/sensors/ftsensor.urdf.xacro" />
+    </xacro:if>
+    <!-- End effector -->
+    <xacro:if value="${has_end_effector}">
+      <xacro:include filename="$(find tiago_description)/urdf/end_effector/end_effector.urdf.xacro" />
+    </xacro:if>
   </xacro:if>
   <!-- Head -->
   <xacro:include filename="$(find tiago_description)/urdf/head/head.urdf.xacro" />
-  <!-- Tools -->
-  <xacro:include filename="$(find pal_urdf_utils)/urdf/deg_to_rad.urdf.xacro" />
   <!-- Materials for visualization -->
   <xacro:include filename="$(find pal_urdf_utils)/urdf/materials.urdf.xacro" />
@@ -137,9 +138,9 @@
   <!-- Torso -->
   <xacro:tiago_torso name="torso" parent="base_link"/>
-  <!-- Arm -->
+  <!-- Arm, FT, EE -->
   <xacro:if value="${has_arm}">
     <!-- Arm -->
     <xacro:tiago_arm name="arm" parent="torso_lift_link" reflect="1" tiago_dual="-1">
-      <origin xyz="0.15505 0.014 -0.151" rpy="0 0 ${-90 * deg_to_rad}" />
+      <origin xyz="${arm_x} ${arm_y} ${arm_z}" rpy="${arm_roll} ${arm_pitch} ${arm_yaw * deg_to_rad}" />
     </xacro:tiago_arm>
     <!-- FT sensor -->
@@ -154,17 +155,4 @@
   <!-- Head -->
   <xacro:head name="head" parent="torso_lift_link"/>
-  <!-- RGBD Laser Link -->
-  <joint name="rgbd_laser_joint" type="fixed">
-    <parent link="base_footprint"/>
-    <child link="rgbd_laser_link"/>
-    <origin xyz="-0.9 0 0" rpy="0 0 0" />
-  </joint>
-  <link name="rgbd_laser_link">
-    <inertial>
-      <origin xyz="0 0 0" rpy="0 0 0"/>
-      <mass value="0.0001" />
-      <inertia ixx="0.0001" ixy="0" ixz="0" iyy="0.0001" iyz="0" izz="0.0001" />
-    </inertial>
-  </link>
   <!-- ROS 2 Control -->
   <xacro:tiago_ros2_control />

File: tiago_description/ros2_control/ros2_control.urdf.xacro (robot description, xacro)
@@ -17,10 +17,17 @@
   <xacro:include filename="$(find tiago_description)/urdf/head/head.ros2_control.xacro" />
   <xacro:include filename="$(find ${base_type}_description)/urdf/wheels/wheel.ros2_control.xacro" />
-  <!-- sensors.ros2_control.xacro should be separated into specific files-->
   <xacro:include filename="$(find ${base_type}_description)/urdf/sensors/sensors.ros2_control.xacro"/>
   <xacro:include filename="$(arg description_calibration_dir)/calibration_constants.urdf.xacro" />
+  <!-- Arm, Wrist, FT, EE -->
   <xacro:if value="${has_arm}">
+    <!-- Arm -->
     <xacro:include filename="$(find tiago_description)/urdf/arm/arm.ros2_control.xacro" />
+    <!-- Wrist -->
     <xacro:include filename="$(find tiago_description)/urdf/arm/wrist.ros2_control.xacro" />
+    <!-- FT sensor -->
+    <xacro:if value="${has_ft_sensor}">
+      <xacro:include filename="$(find tiago_description)/urdf/sensors/ftsensor.ros2_control.xacro"/>
+    </xacro:if>
+    <!-- End effector -->
     <xacro:if value="${end_effector == 'pal-gripper'}">
       <xacro:include filename="$(find pal_gripper_description)/urdf/gripper.ros2_control.xacro" />
@@ -32,7 +39,4 @@
       <xacro:include filename="$(find pal_robotiq_description)/urdf/robotiq.ros2_control.xacro" />
     </xacro:if>
-  </xacro:if>
-  <xacro:if value="${has_ft_sensor}">
-    <xacro:include filename="$(find tiago_description)/urdf/sensors/ftsensor.ros2_control.xacro"/>
   </xacro:if>
   <!-- MACRO DEFINITION-->
@@ -66,5 +70,5 @@
       <!-- Torso -->
       <xacro:ros2_control_torso name="torso_lift" reduction="1.0" />
-      <!-- Arm -->
+      <!-- Arm, Wrist, FT, EE -->
       <xacro:if value="${has_arm}">
         <!-- Arm -->

File: tiago_description/ros2_control/transmissions.urdf.xacro (robot description, xacro)
@@ -13,4 +13,5 @@
  -->
 <robot xmlns:xacro="http://ros.org/wiki/xacro">
+  <!-- MACRO DEFINITION -->
   <xacro:macro name="tiago_simple_transmission" params="name reduction:=1.0 offset_value:=0.0">
     <transmission name="${name}_trans">

File: tiago_description/urdf/arm/arm.urdf.xacro (robot description, xacro)
@@ -13,7 +13,4 @@
  -->
 <robot xmlns:xacro="http://ros.org/wiki/xacro">
-  <!-- INCLUDES -->
-  <xacro:include filename="$(find pal_urdf_utils)/urdf/deg_to_rad.urdf.xacro" />
-  <xacro:include filename="$(find tiago_description)/urdf/arm/wrist.urdf.xacro" />
   <!-- PROPERTIES -->
   <xacro:property name="arm_friction" value="1.0" />
@@ -34,4 +31,7 @@
     <xacro:property name="tool_link_z_offset" value="${ 0.046 if has_ft_sensor else 0.0573 }"/>
   </xacro:if>
+  <!-- INCLUDES -->
+  <xacro:include filename="$(find pal_urdf_utils)/urdf/deg_to_rad.urdf.xacro" />
+  <xacro:include filename="$(find tiago_description)/urdf/arm/wrist.urdf.xacro" />
   <!-- MACRO DEFINITION-->
   <xacro:macro name="tiago_arm" params="name parent reflect tiago_dual *origin">

File: tiago_description/urdf/arm/wrist.urdf.xacro (robot description, xacro)
@@ -13,6 +13,4 @@
  -->
 <robot xmlns:xacro="http://ros.org/wiki/xacro">
-  <!-- INCLUDES -->
-  <xacro:include filename="$(find pal_urdf_utils)/urdf/deg_to_rad.urdf.xacro" />
   <!-- PROPERTIES -->
   <xacro:property name="wrist_friction" value="1.0" />
@@ -31,4 +29,6 @@
     <xacro:property name="wrist_6_range" value="81"/>
   </xacro:if>
+  <!-- INCLUDES -->
+  <xacro:include filename="$(find pal_urdf_utils)/urdf/deg_to_rad.urdf.xacro" />
   <!-- MACRO DEFINITION -->
   <xacro:macro name="wrist" params="name parent reflect">

File: tiago_description/urdf/end_effector/end_effector.urdf.xacro (robot description, xacro)
@@ -17,11 +17,11 @@
   <xacro:include filename="$(find pal_hey5_description)/urdf/pal_hey5_hand.urdf.xacro" />
   <xacro:if value="${end_effector == 'pal-gripper'}">
-    <xacro:include filename="$(find pal_gripper_description)/urdf/gripper.ros2_control.xacro" />
+    <xacro:include filename="$(find pal_gripper_description)/urdf/gripper.urdf.xacro" />
   </xacro:if>
-  <xacro:if value="${end_effector == 'pal-hey5'}">
-    <xacro:include filename="$(find pal_hey5_description)/urdf/pal_hey5.ros2_control.xacro" />
+  <xacro:if value="${end_effector == 'robotiq-2f-85'}">
+    <xacro:include filename="$(find pal_robotiq_description)/urdf/robotiq_85_gripper.urdf.xacro" />
   </xacro:if>
-  <xacro:if value="${end_effector in ['robotiq-2f-85', 'robotiq-2f-140']}">
-    <xacro:include filename="$(find pal_robotiq_description)/urdf/robotiq.ros2_control.xacro" />
+  <xacro:if value="${end_effector == 'robotiq-2f-140'}">
+    <xacro:include filename="$(find pal_robotiq_description)/urdf/robotiq_140_gripper.urdf.xacro" />
   </xacro:if>
   <!-- MACRO DEFINITION -->

File: tiago_description/urdf/sensors/ftsensor.gazebo.xacro (robot description, xacro)
@@ -13,4 +13,5 @@
  -->
 <robot xmlns:xacro="http://ros.org/wiki/xacro">
+  <!-- MACRO DEFINITION -->
   <xacro:macro name="force_torque_sensor_gazebo" params="name update_rate">
     <gazebo reference="${name}_joint">

Commit message: Module, joy config and restored support for tiago dual

File: tiago_description/robots/tiago.urdf.xacro (robot description, xacro)
@@ -141,5 +141,5 @@
   <xacro:if value="${has_arm}">
     <!-- Arm -->
-    <xacro:tiago_arm name="arm" parent="torso_lift_link" reflect="1" tiago_dual="-1">
+    <xacro:tiago_arm name="arm" parent="torso_lift_link" wrist_model="${wrist_model}" has_ft_sensor="${has_ft_sensor}" reflect="1" tiago_dual="-1">
       <origin xyz="${arm_x} ${arm_y} ${arm_z}" rpy="${arm_roll} ${arm_pitch} ${arm_yaw * deg_to_rad}" />
     </xacro:tiago_arm>
@@ -150,5 +150,5 @@
     <!-- End effector -->
     <xacro:if value="${has_end_effector}">
-      <xacro:tiago_end_effector name="${end_effector_name}" parent="${end_effector_link}" reflect="1"/>
+      <xacro:tiago_end_effector name="${end_effector_name}" parent="${end_effector_link}" end_effector="${end_effector}" reflect="1"/>
     </xacro:if>
   </xacro:if>

File: tiago_description/ros2_control/ros2_control.urdf.xacro (robot description, xacro)
@@ -18,5 +18,5 @@
   <xacro:include filename="$(find ${base_type}_description)/urdf/wheels/wheel.ros2_control.xacro" />
   <xacro:include filename="$(find ${base_type}_description)/urdf/sensors/sensors.ros2_control.xacro"/>
-  <xacro:include filename="$(arg description_calibration_dir)/calibration_constants.urdf.xacro" />
+  <xacro:include filename="${description_calibration_dir}/calibration_constants.urdf.xacro" />
   <!-- Arm, Wrist, FT, EE -->
   <xacro:if value="${has_arm}">
@@ -42,5 +42,5 @@
   <!-- MACRO DEFINITION-->
   <xacro:macro name="tiago_ros2_control">
-    <!-- ROS 2 config-->
+    <!-- ROS 2 control config-->
     <ros2_control name="ros2_control_tiago_system" type="system">
       <!-- Execution env config -->

File: tiago_description/urdf/arm/arm.urdf.xacro (robot description, xacro)
@@ -25,15 +25,16 @@
   <xacro:property name="arm_4_max_effort" value="26" />
   <xacro:property name="arm_eps" value="${0.00 if no_safety_eps else 0.07}"/>
-  <xacro:if value="${wrist_model == 'wrist-2010'}">
-    <xacro:property name="tool_link_z_offset" value="0.046"/>
-  </xacro:if>
-  <xacro:if value="${wrist_model == 'wrist-2017'}">
-    <xacro:property name="tool_link_z_offset" value="${ 0.046 if has_ft_sensor else 0.0573 }"/>
-  </xacro:if>
   <!-- INCLUDES -->
   <xacro:include filename="$(find pal_urdf_utils)/urdf/deg_to_rad.urdf.xacro" />
   <xacro:include filename="$(find tiago_description)/urdf/arm/wrist.urdf.xacro" />
   <!-- MACRO DEFINITION-->
-  <xacro:macro name="tiago_arm" params="name parent reflect tiago_dual *origin">
+  <xacro:macro name="tiago_arm" params="name parent reflect wrist_model has_ft_sensor tiago_dual *origin">
+    <!-- Param related properties -->
+    <xacro:if value="${wrist_model == 'wrist-2010'}">
+      <xacro:property name="tool_link_z_offset" value="0.046"/>
+    </xacro:if>
+    <xacro:if value="${wrist_model == 'wrist-2017'}">
+      <xacro:property name="tool_link_z_offset" value="${ 0.046 if has_ft_sensor else 0.0573 }"/>
+    </xacro:if>
     <!-- Shoulder -->
     <link name="${name}_1_link">
@@ -197,5 +198,5 @@
     </gazebo>
     <!-- Wrist -->
-    <xacro:wrist name="${name}" parent="${name}_4_link" reflect="${reflect}"/>
+    <xacro:wrist name="${name}" parent="${name}_4_link" wrist_model="${wrist_model}" reflect="${reflect}"/>
     <!-- Tool -->
     <link name="${name}_tool_link">

File: tiago_description/urdf/arm/wrist.urdf.xacro (robot description, xacro)
@@ -23,14 +23,15 @@
   <xacro:property name="wrist_3_max_effort" value="6.6" />
   <xacro:property name="wrist_eps" value="${0.00 if no_safety_eps else 0.02}"/>
-  <xacro:if value="${wrist_model == 'wrist-2010'}">
-    <xacro:property name="wrist_6_range" value="${ 81 if has_ft_sensor else 90 }"/>
-  </xacro:if>
-  <xacro:if value="${wrist_model == 'wrist-2017'}">
-    <xacro:property name="wrist_6_range" value="81"/>
-  </xacro:if>
   <!-- INCLUDES -->
   <xacro:include filename="$(find pal_urdf_utils)/urdf/deg_to_rad.urdf.xacro" />
   <!-- MACRO DEFINITION -->
-  <xacro:macro name="wrist" params="name parent reflect">
+  <xacro:macro name="wrist" params="name parent wrist_model reflect">
+    <!-- Param dependant properties -->
+    <xacro:if value="${wrist_model == 'wrist-2010'}">
+      <xacro:property name="wrist_6_range" value="${ 81 if has_ft_sensor else 90 }"/>
+    </xacro:if>
+    <xacro:if value="${wrist_model == 'wrist-2017'}">
+      <xacro:property name="wrist_6_range" value="81"/>
+    </xacro:if>
     <!-- Wrist-->
     <link name="${name}_5_link">

File: tiago_description/urdf/end_effector/end_effector.urdf.xacro (robot description, xacro)
@@ -16,15 +16,16 @@
   <xacro:include filename="$(find pal_urdf_utils)/urdf/deg_to_rad.urdf.xacro" />
   <xacro:include filename="$(find pal_hey5_description)/urdf/pal_hey5_hand.urdf.xacro" />
-  <xacro:if value="${end_effector == 'pal-gripper'}">
-    <xacro:include filename="$(find pal_gripper_description)/urdf/gripper.urdf.xacro" />
-  </xacro:if>
-  <xacro:if value="${end_effector == 'robotiq-2f-85'}">
-    <xacro:include filename="$(find pal_robotiq_description)/urdf/robotiq_85_gripper.urdf.xacro" />
-  </xacro:if>
-  <xacro:if value="${end_effector == 'robotiq-2f-140'}">
-    <xacro:include filename="$(find pal_robotiq_description)/urdf/robotiq_140_gripper.urdf.xacro" />
-  </xacro:if>
   <!-- MACRO DEFINITION -->
-  <xacro:macro name="tiago_end_effector" params="name parent reflect tiago_dual:=false">
+  <xacro:macro name="tiago_end_effector" params="name parent reflect end_effector tiago_dual:=false">
+    <!-- Param dependant includes -->
+    <xacro:if value="${end_effector == 'pal-gripper'}">
+      <xacro:include filename="$(find pal_gripper_description)/urdf/gripper.urdf.xacro" />
+    </xacro:if>
+    <xacro:if value="${end_effector == 'robotiq-2f-85'}">
+      <xacro:include filename="$(find pal_robotiq_description)/urdf/robotiq_85_gripper.urdf.xacro" />
+    </xacro:if>
+    <xacro:if value="${end_effector == 'robotiq-2f-140'}">
+      <xacro:include filename="$(find pal_robotiq_description)/urdf/robotiq_140_gripper.urdf.xacro" />
+    </xacro:if>
     <!-- PAL Gripper -->
     <xacro:if value="${end_effector == 'pal-gripper'}">

Commit message: Suggested changed

File: tiago_description/robots/tiago.urdf.xacro (robot description, xacro)
@@ -27,4 +27,6 @@
   <!-- no-laser, hokuyo, sick-551, sick-561, sick-571-->
   <xacro:arg name="laser_model" default="sick-571"/>
+  <!-- false, true -->
+  <xacro:arg name="has_screen" default="false"/>
   <!-- no-arm, tiago-arm -->
   <xacro:arg name="arm_model" default="tiago-arm"/>
@@ -58,4 +60,5 @@
   <xacro:property name="camera_model" value="$(arg camera_model)" />
   <xacro:property name="has_thermal_camera" default="$(arg has_thermal_camera)"/>
+  <xacro:property name="has_screen" value="$(arg has_screen)" />
   <xacro:property name="no_safety_eps" value="$(arg no_safety_eps)" />
   <!-- HW configuration check -->

Commit message: Changed arm_model to arm_type in the URDF

File: tiago_description/robots/tiago.urdf.xacro (robot description, xacro)
@@ -30,5 +30,5 @@
   <xacro:arg name="has_screen" default="false"/>
   <!-- no-arm, tiago-arm -->
-  <xacro:arg name="arm_model" default="tiago-arm"/>
+  <xacro:arg name="arm_type" default="tiago-arm"/>
   <!-- no-ft-sensor, schunk-ft -->
   <xacro:arg name="ft_sensor" default="schunk-ft"/>
@@ -54,5 +54,5 @@
   <xacro:property name="base_type" value="$(arg base_type)" />
   <xacro:property name="laser_model" value="$(arg laser_model)" />
-  <xacro:property name="arm_model" value="$(arg arm_model)" />
+  <xacro:property name="arm_type" value="$(arg arm_type)" />
   <xacro:property name="ft_sensor" value="$(arg ft_sensor)" />
   <xacro:property name="wrist_model" value="$(arg wrist_model)" />
@@ -69,5 +69,5 @@
     <xacro:wrong_laser_model/>
   </xacro:if>
-  <xacro:if value="${arm_model not in ['no-arm', 'tiago-arm']}">
+  <xacro:if value="${arm_type not in ['no-arm', 'tiago-arm']}">
     <xacro:wrong_arm/>
   </xacro:if>
@@ -85,5 +85,5 @@
   </xacro:if>
   <!-- HW configuration helpers-->
-  <xacro:property name="has_arm" value="${arm_model != 'no-arm'}"/>
+  <xacro:property name="has_arm" value="${arm_type != 'no-arm'}"/>
   <xacro:property name="has_ft_sensor" value="${ft_sensor != 'no-ft-sensor'}"/>
   <xacro:property name="has_end_effector" value="${end_effector != 'no-end-effector'}"/>

Commit message: add missing argument is_public_sim

File: tiago_description/robots/tiago.urdf.xacro (robot description, xacro)
@@ -50,4 +50,5 @@
   <xacro:arg name="is_multiple" default="false"/>
   <xacro:arg name="namespace" default=""/>
+  <xacro:arg name="is_public_sim" default="false"/>
   <!-- PROPERTIES -->
   <!-- HW configuration -->
@@ -103,4 +104,5 @@
   <xacro:property name="is_multiple" value="$(arg is_multiple)" />
   <xacro:property name="namespace" value="$(arg namespace)" />
+  <xacro:property name="is_public_sim" value="$(arg is_public_sim)" />
   <!-- INCLUDES -->
   <!-- Tools -->
