Commit message: Fix distance of from the arm_7_link to arm_tool_link and the ft_sensor link placement

File: tiago_description/urdf/arm/arm.urdf.xacro (robot description, xacro)
@@ -35,5 +35,5 @@
     </xacro:if>
     <xacro:if value="${wrist_model == 'wrist-2017'}">
-      <xacro:property name="tool_link_z_offset" value="${ 0.046 if has_ft_sensor else 0.0573 }"/>
+      <xacro:property name="tool_link_z_offset" value="${ 0.051875 if has_ft_sensor else 0.0615 }"/>
     </xacro:if>
     <!-- Shoulder -->

File: tiago_description/urdf/sensors/ftsensor.urdf.xacro (robot description, xacro)
@@ -20,6 +20,6 @@
     <link name="${name}_ft_link">
       <inertial>
-        <mass value="0.1" />
-        <inertia ixx="0.0" ixy="0.0" ixz="0.0" iyy="0.0" iyz="0.0" izz="0.0" />
+        <mass value="0.095000" />
+        <inertia ixx="0.000016" ixy="-0.000001" ixz="0.0" iyy="0.000015" iyz="0.0" izz="0.000027" />
       </inertial>
       <visual>
@@ -40,5 +40,5 @@
       <parent link="${parent}" />
       <child link="${name}_ft_link" />
-      <origin xyz="${0.0157*0.5} 0 0" rpy="${90.0 * deg_to_rad} 0 ${90.0 * deg_to_rad}" />
+      <origin xyz="${0.0157*0.5 + 0.001525} 0 0" rpy="${90.0 * deg_to_rad} 0 ${90.0 * deg_to_rad}" />
     </joint>
     <!-- FT tool -->
@@ -65,5 +65,5 @@
       <parent link="${name}_ft_link" />
       <child link="${name}_ft_tool_link" />
-      <origin xyz="0 0 ${0.0157*0.5 + 0.00975*0.5}" rpy="${-90.0 * deg_to_rad} ${-90.0 * deg_to_rad} 0" />
+      <origin xyz="0 0 ${0.0157*0.5 + 0.00975*0.5 -0.001525}" rpy="${-90.0 * deg_to_rad} ${-90.0 * deg_to_rad} 0" />
     </joint>
     <!-- Gazebo config-->

Commit message: Fix distances for old wrist + change default wrist + typo

File: tiago_description/urdf/arm/arm.urdf.xacro (robot description, xacro)
@@ -32,5 +32,5 @@
     <!-- Param related properties -->
     <xacro:if value="${wrist_model == 'wrist-2010'}">
-      <xacro:property name="tool_link_z_offset" value="0.046"/>
+      <xacro:property name="tool_link_z_offset" value="${ 0.056873 if has_ft_sensor else 0.0518 }"/>
     </xacro:if>
     <xacro:if value="${wrist_model == 'wrist-2017'}">

File: tiago_description/urdf/sensors/ftsensor.urdf.xacro (robot description, xacro)
@@ -65,5 +65,5 @@
       <parent link="${name}_ft_link" />
       <child link="${name}_ft_tool_link" />
-      <origin xyz="0 0 ${0.0157*0.5 + 0.00975*0.5 -0.001525}" rpy="${-90.0 * deg_to_rad} ${-90.0 * deg_to_rad} 0" />
+      <origin xyz="0 0 ${0.0157*0.5 + 0.00975*0.5 - 0.001525}" rpy="${-90.0 * deg_to_rad} ${-90.0 * deg_to_rad} 0" />
     </joint>
     <!-- Gazebo config-->
